Commit message: Add files via upload
masse filer, alt som må huskes er at launch filene og urdf filen for den andre sonaren jeg lagde er ikke her. Derimot burde være lett å implementere.

File: urdf/tms_second.xacro (robot description, xacro)
@@ -3,5 +3,5 @@
   <!-- Necessary for sonar to work -->
   <xacro:arg name="namespace" default="tms"/>
-  <xacro:include filename="$(find uuv_sensor_ros_plugins)/urdf/sonar_snippets.xacro" />
+  <!-- <xacro:include filename="$(find uuv_sensor_ros_plugins)/urdf/sonar_snippets.xacro" /> -->
   <!-- Necessary for thruster_macro to work -->
   <xacro:include filename="$(find deep_ocean)/urdf/actuators.xacro" />
@@ -13,5 +13,5 @@
   <xacro:property name="fluid_density" value="1028"/>
   <!-- Scaling Factor for the TMS. Greater size means it's easier to dock -->
-  <xacro:property name="scale_factor" value="1"/> <!-- Change this to scale up/down -->
+  <xacro:property name="scale_factor" value="1.0"/> <!-- Change this to scale up/down -->
   <!-- Original Dimensions of the TMS -->
   <xacro:property name="size_x_orig" value="1.64"/>
@@ -23,5 +23,5 @@
   <xacro:property name="size_z" value="${size_z_orig * scale_factor}"/>
   <!-- Mass (Scaled) -->
-  <xacro:property name="mass" value="${550 * (scale_factor * scale_factor * scale_factor)}"/>
+  <xacro:property name="mass" value="${550.0 * (scale_factor * scale_factor * scale_factor)}"/>
   <!-- Volume (to ensure neutral buoyancy) -->
   <xacro:property name="volume" value="${mass / fluid_density}"/>
@@ -35,5 +35,5 @@
     <inertial>
       <mass value="${mass}"/>
-      <origin xyz="0 0 0" rpy="0 0 3.14159"/>5
+      <origin xyz="0 0 0" rpy="0 0 3.14159"/>
       <inertia ixx="${ixx}" ixy="0.0" ixz="0.0" iyy="${iyy}" iyz="0.0" izz="${izz}"/>
     </inertial>
@@ -113,6 +113,120 @@
   </xacro:thruster_macro>
   <!-- initilizing Sonar macro -->
-  <xacro:forward_multibeam_sonar_m450_130 namespace="$(arg namespace)" parent_link="$(arg namespace)/base_link">
+  <!-- bruker denne som referanse til hjemmebygd sonar -->
+  <!-- <xacro:forward_multibeam_sonar_m450_130 namespace="$(arg namespace)" parent_link="$(arg namespace)/base_link">
     <origin xyz="-0.9 0 1.02" rpy="0 0 3.14159"/>
-  </xacro:forward_multibeam_sonar_m450_130>
+  </xacro:forward_multibeam_sonar_m450_130> -->
+<!-- kanskje prøve å etterligne denne https://waterlinked.com/shop/wl-21045-2-sonar-3d-15-689 -->
+  <link name= "depth_camera_link">
+      <visual>
+          <geometry>
+              <box size= "0.04 0.12 0.08" />
+          </geometry>
+          <material name= "red" >
+              <color rgba= "1 0 0 1" />
+          </material>
+      </visual>
+      <inertial>
+          <!-- <mass value= "0.39" /> -->
+          <mass value= "0.0" />
+          <origin xyz= "0 0 0" />
+          <inertia ixx= "0.1" ixy= "0.0" ixz= "0.0" iyy= "0.1" iyz= "0.0" izz= "0.1" />
+      </inertial>
+      <collision>
+          <geometry>
+              <box size= "0.04 0.12 0.08" />
+          </geometry>
+      </collision>
+  </link>
+    <joint name= "depth_camera_joint" type= "fixed">
+        <parent link= "$(arg namespace)/base_link" />
+        <child link= "depth_camera_link" />
+        <!-- <origin xyz= "0.55 0 3 " rpy= "0 0 0"/> -->
+        <origin xyz="-0.8 0 1.02" rpy="0 0 3.14159"/>
+    </joint>
+  <!-- optical link and joint for rviz -->
+  <link name= "depth_camera_optical_link"></link>
+  <joint name= "depth_camera_optical_joint" type= "fixed">
+      <parent link= "depth_camera_link" />
+      <child link= "depth_camera_optical_link" />
+      <origin xyz= "0 0 0 " rpy= "-1.57 0 -1.57"/>
+  </joint>
+  <gazebo reference= "depth_camera_link">
+      <material>Gazebo/Red</material>
+      <sensor name= "depth_camera_link" type= "depth">
+          <visualize>true</visualize>
+          <updateRate>10</updateRate>
+          <camera>
+              <horizontal_fov>1.57</horizontal_fov>
+              <vertical_fov>0.698</vertical_fov>
+              <image>
+                  <width>160</width>
+                  <height>100</height>
+              </image>
+              <clip>
+                  <near>0.1</near>
+                  <far>5.0</far>
+              </clip>
+          </camera>
+          <plugin name="depth_camera_sensor" filename="libgazebo_ros_openni_kinect.so">
+              <cameraName>depth_camera</cameraName>
+              <frameName>$(arg namespace)/depth_camera_optical_link</frameName>
+              <alwaysOn>true</alwaysOn>
+              <pointCloudTopicName>points</pointCloudTopicName>
+              <imageTopicName>rgb/image_raw</imageTopicName>
+              <depthImageTopicName>depth/image_raw</depthImageTopicName>
+              <cameraInfoTopicName>rgb/camera_info</cameraInfoTopicName>
+              <depthImageCameraInfoTopicName>depth/camera_info</depthImageCameraInfoTopicName>
+              <!-- <baseline>0.1</baseline> -->
+          </plugin>
+      </sensor>
+  </gazebo>
+  <!-- imu sensor -->
+  <link name= "imu_link">
+      <visual>
+          <geometry>
+              <box size= "0.01 0.01 0.01" />
+          </geometry>
+          <material name= "red" >
+              <color rgba= "1 0 0 1" />
+          </material>
+      </visual>
+      <inertial>
+          <!-- <mass value= "0.39" /> -->
+          <mass value= "0.0" />
+          <origin xyz= "0 0 0" />
+          <inertia ixx= "0.1" ixy= "0.0" ixz= "0.0" iyy= "0.1" iyz= "0.0" izz= "0.1" />
+      </inertial>
+      <collision>
+          <geometry>
+              <box size= "0.01 0.01 0.01" />
+          </geometry>
+      </collision>
+  </link>
+  <joint name= "imu_joint" type= "fixed">
+      <parent link= "$(arg namespace)/base_link" />
+      <child link= "imu_link" />
+      <!-- <origin xyz= "0.55 0 3 " rpy= "0 0 0"/> -->
+      <origin xyz="0 0 0.81" rpy="0 0 0"/>
+  </joint>
+  <gazebo reference="imu_link">
+    <gravity>true</gravity>
+    <sensor name="imu_sensor" type="imu">
+      <always_on>true</always_on>
+      <update_rate>10</update_rate>
+      <visualize>true</visualize>
+      <topic>__default_topic__</topic>
+      <plugin filename="libgazebo_ros_imu_sensor.so" name="imu_plugin">
+        <topicName>imu</topicName>
+        <bodyName>imu_link</bodyName>
+        <updateRateHZ>10.0</updateRateHZ>
+        <gaussianNoise>0.0</gaussianNoise>
+        <xyzOffset>0 0 0</xyzOffset>
+        <rpyOffset>0 0 0</rpyOffset>
+        <frameName>imu_link</frameName>
+        <initialOrientationAsReference>false</initialOrientationAsReference>
+      </plugin>
+      <pose>0 0 0 0 0 0</pose>
+    </sensor>
+  </gazebo>
 </robot>
