Commit message: Add files via upload

File: urdf/rov.xacro (robot description, xacro)
@@ -1,4 +1,8 @@
 <?xml version="1.0"?>
 <robot name="rov" xmlns:xacro="http://www.ros.org/wiki/xacro">
+  <xacro:arg name="namespace" default="rov"/>
+  <xacro:include filename="$(find deep_ocean)/urdf/actuators.xacro" />
+  <xacro:include filename="$(find uuv_descriptions)/urdf/common.urdf.xacro" />
+  <xacro:include filename="$(find uuv_gazebo_ros_plugins)/urdf/thruster_snippets.xacro" />
     <!-- Fluid Density of Water (kg/m³) -->
     <xacro:property name="fluid_density" value="1028"/>
@@ -18,5 +22,5 @@
     <xacro:property name="izz" value="${(1/12) * mass * (size_x * size_x + size_y * size_y)}"/>
     <!-- Define Base Link -->
-    <link name="base_link">
+    <link name="$(arg namespace)/base_link">
         <inertial>
             <mass value="${mass}"/>
@@ -58,5 +62,5 @@
         </link>
         <joint name="${thruster_name}_joint" type="fixed">
-            <parent link="base_link"/>
+            <parent link="$(arg namespace)/base_link"/>
             <child link="${thruster_name}"/>
             <origin xyz="${x} ${y} ${z}" rpy="${roll} ${pitch} ${yaw}"/>
@@ -71,4 +75,26 @@
     <xacro:thruster thruster_name="thruster_6" x="-0.3381" y="0.15606" z="0.38038" roll="1.5708" pitch="0" yaw="-0.6981"/>
     <xacro:thruster thruster_name="thruster_7" x="-0.002266" y="-0.39991" z="0.70723" roll="-0.3491" pitch="0" yaw="0"/>
+    <!-- All of them are 90 degrees wrong for the moment -->
+  <!--xacro:thruster_macro namespace="$(arg namespace)" thruster_id="0">
+    <origin xyz="0.22357 -0.56374 0.38038" rpy="1.5708 0 -0.6981"/>
+  </xacro:thruster_macro>
+  <xacro:thruster_macro namespace="$(arg namespace)" thruster_id="1">
+    <origin xyz="0.3381 0.15606 0.38038" rpy="1.5708 0 0.6981"/>
+  </xacro:thruster_macro>
+  <xacro:thruster_macro namespace="$(arg namespace)" thruster_id="2">
+    <origin xyz="0.30171 0.060821 0.70723" rpy="0.1745 -0.3491 0"/>
+  </xacro:thruster_macro>
+  <xacro:thruster_macro namespace="$(arg namespace)" thruster_id="3">
+    <origin xyz="-0.22357 -0.56374 0.38038" rpy="1.5708 0 0.6981"/>
+  </xacro:thruster_macro>
+  <xacro:thruster_macro namespace="$(arg namespace)" thruster_id="4">
+    <origin xyz="-0.3017 0.060821 0.70723" rpy="0.1745 0.3491 0"/>
+  </xacro:thruster_macro>
+  <xacro:thruster_macro namespace="$(arg namespace)" thruster_id="5">
+    <origin xyz="-0.3381 0.15606 0.38038" rpy="1.5708 0 -0.6981"/>
+  </xacro:thruster_macro>
+  <xacro:thruster_macro namespace="$(arg namespace)" thruster_id="6">
+    <origin xyz="-0.002266 -0.39991 0.70723" rpy="-0.3491 0 0"/>
+  </xacro:thruster_macro-->
     <gazebo>
         <plugin name="uuv_plugin" filename="libuuv_underwater_object_ros_plugin.so">
@@ -76,5 +102,5 @@
             <flow_velocity_topic>hydrodynamics/current_velocity</flow_velocity_topic>
             <debug>0</debug>
-            <link name="base_link">
+            <link name="$(arg namespace)/base_link">
                 <neutrally_buoyant>1</neutrally_buoyant>  <!-- Ensures mass and volume decide float/sink -->
                 <volume>${volume}</volume>

File: urdf/tms.xacro (robot description, xacro)
@@ -53,4 +53,16 @@
     </collision>
   </link>
+  <!-- An attempt to restrict movement in z axis -->
+  <!--joint name="xy_plane_joint" type="planar">
+    <parent link="world"/>
+    <child link="base_link"/>
+    <axis xyz="1 0 0"/>
+    <axis2 xyz="0 1 0"/>
+  </joint>
+  <joint name="yaw_joint" type="continuous">
+    <parent link="world"/>
+    <child link="base_link"/>
+    <axis xyz="0 0 1"/>
+  </joint-->
   <gazebo>
     <plugin name="uuv_plugin" filename="libuuv_underwater_object_ros_plugin.so">
@@ -103,8 +115,8 @@
   <!-- Initilizing thruster macro, might use another macro to achieve thrusters -->
   <xacro:thruster_macro namespace="$(arg namespace)" thruster_id="0">
-    <origin xyz="0.7650895 0.467385 0.528822" rpy="0 0 ${pi/2}"/>
+    <origin xyz="0.6650895 0.367385 0.828822" rpy="0 0 ${3*pi/4}"/>
   </xacro:thruster_macro>
   <xacro:thruster_macro namespace="$(arg namespace)" thruster_id="1">
-    <origin xyz="0.765895 -0.467385 0.528822" rpy="0 0 ${-pi/2}"/>
+    <origin xyz="0.665895 -0.367385 0.828822" rpy="0 0 ${-3*pi/4}"/>
   </xacro:thruster_macro>
   <!-- initilizing Sonar macro -->

Commit message: Add files via upload

File: urdf/rov.xacro (robot description, xacro)
@@ -2,4 +2,7 @@
 <robot name="rov" xmlns:xacro="http://www.ros.org/wiki/xacro">
   <xacro:arg name="namespace" default="rov"/>
+    <!-- Necessary for sensors -->
+    <xacro:include filename="$(find deep_ocean)/urdf/sonar_snippets.xacro" />
+    <!-- <xacro:include filename="$(find uuv_sensor_ros_plugins)/urdf/sensor_snippets.xacro"/> -->
     <!-- Necessary for thrusters -->
     <xacro:include filename="$(find deep_ocean)/urdf/actuators.xacro" />
@@ -68,4 +71,12 @@
   </xacro:thruster_macro>
   <xacro:default_joint_state_publisher namespace="$(arg namespace)" update_rate="50"/>
+    <!-- initilizing Sonar macro -->
+  <xacro:forward_multibeam_sonar_m450_130 namespace="$(arg namespace)" parent_link="$(arg namespace)/base_link">
+    <origin xyz="0.63 0 0.63" rpy="0 0 0"/>
+  </xacro:forward_multibeam_sonar_m450_130>
+    <!-- mounting camera -->
+  <!--xacro:default_camera namespace="$(arg namespace)" parent_link="$(arg namespace)/base_link" suffix="">
+    <origin xyz="0.63 0 0.4" rpy="0 0.6 0"/>
+  </xacro:default_camera-->
     <gazebo>
         <plugin name="uuv_plugin" filename="libuuv_underwater_object_ros_plugin.so">

File: urdf/sonar_snippets.xacro (robot description, xacro)
@@ -48,5 +48,5 @@
   </xacro:macro>
   <!-- Inspired by m450-130: http://www.blueview.com/products/2d-imaging-sonar/m900-series/ -->
-  <xacro:macro name="forward_multibeam_sonar_m450_130" params="namespace parent_link *origin">
+  <xacro:macro name="forward_multibeam_sonar_m450_130" params="namespace parent_link visualize:=true *origin">
     <xacro:multibeam_sonar
       namespace="${namespace}"
@@ -54,5 +54,5 @@
       parent_link="${parent_link}"
       topic="sonar"
-      mass="0.015"
+      mass="0.0001"
       update_rate="25"
       samples="100"
@@ -61,5 +61,6 @@
       range_max="5.0"
       range_stddev="0.027"
-      mesh="">
+      mesh=""
+      visualize="${visualize}">
       <inertia ixx="0.00001" ixy="0.0" ixz="0.0" iyy="0.00001" iyz="0.0" izz="0.00001" />
       <xacro:insert_block name="origin" />
@@ -96,5 +97,5 @@
   <xacro:macro name="multibeam_sonar"
     params="namespace suffix parent_link topic mass update_rate
-      samples fov range_min range_max range_stddev mesh
+      samples fov range_min range_max range_stddev mesh visualize
       *inertia *origin *visual">
     <!-- Sensor link -->
@@ -112,11 +113,11 @@
     <parent link="${parent_link}" />
     <child link="${namespace}/sonar${suffix}_link" />
-    <limit upper="0.13" lower="0.13" effort="0" velocity="0" />
-    <axis xyz="0 1 0"/>
+    <limit upper="0" lower="0" effort="0" velocity="0" />
+    <axis xyz="1 0 0"/>
   </joint>
   <gazebo reference="${namespace}/sonar${suffix}_link">
     <sensor type="gpu_ray" name="sonar${suffix}">
       <pose>0 0 0 0 0 0</pose>
-      <visualize>true</visualize>
+      <visualize>${visualize}</visualize>
       <update_rate>${update_rate}</update_rate>
       <ray>

File: urdf/thruster_snippets.xacro (robot description, xacro)
@@ -84,5 +84,5 @@
     </joint>
     <link name="${namespace}/thruster_${thruster_id}">
-      <xacro:box_inertial x="0" y="0" z="0" mass="0.001">
+      <xacro:box_inertial x="0" y="0" z="0" mass="0.000000001">
         <origin xyz="0 0 0" rpy="0 0 0"/>
       </xacro:box_inertial>

File: urdf/tms_second.xacro (robot description, xacro)
@@ -36,5 +36,5 @@
     <inertial>
       <mass value="${mass}"/>
-      <origin xyz="0 0 0" rpy="0 0 3.14159"/>
+      <origin xyz="0 0 0" rpy="0 0 3.14159"/>5
       <inertia ixx="${ixx}" ixy="0.0" ixz="0.0" iyy="${iyy}" iyz="0.0" izz="${izz}"/>
     </inertial>
@@ -107,4 +107,81 @@
     </plugin>
   </gazebo>
+  <xacro:default_joint_state_publisher namespace="$(arg namespace)" update_rate="50"/>
+  <!-- Initilizing thruster macro, might use another macro to achieve thrusters -->
+  <xacro:thruster_macro namespace="$(arg namespace)" thruster_id="0" mesh_scale="1">
+    <origin xyz="0.6650895 0.367385 0.828822" rpy="0 0 ${3*pi/4}"/>
+  </xacro:thruster_macro>
+  <xacro:thruster_macro namespace="$(arg namespace)" thruster_id="1" mesh_scale="1">
+    <origin xyz="0.665895 -0.367385 0.828822" rpy="0 0 ${-3*pi/4}"/>
+  </xacro:thruster_macro>
+  <!-- initilizing Sonar macro -->
+  <!--xacro:forward_multibeam_sonar_m450_130 namespace="$(arg namespace)" parent_link="$(arg namespace)/base_link" visualize="$(arg visualize)">
+    <origin xyz="-0.9 0 0.97" rpy="0 0 3.14159"/>
+  </xacro:forward_multibeam_sonar_m450_130-->
+<!-- kanskje prøve å etterligne denne https://waterlinked.com/shop/wl-21045-2-sonar-3d-15-689 -->
+  <link name= "depth_camera_link">
+      <visual>
+          <geometry>
+              <box size= "0.04 0.12 0.08" />
+          </geometry>
+          <material name= "red" >
+              <color rgba= "1 0 0 1" />
+          </material>
+      </visual>
+      <inertial>
+          <!-- <mass value= "0.39" /> -->
+          <mass value= "0.0" />
+          <origin xyz= "0 0 0" />
+          <inertia ixx= "0.1" ixy= "0.0" ixz= "0.0" iyy= "0.1" iyz= "0.0" izz= "0.1" />
+      </inertial>
+      <collision>
+          <geometry>
+              <box size= "0.04 0.12 0.08" />
+          </geometry>
+      </collision>
+  </link>
+    <joint name= "depth_camera_joint" type= "fixed">
+        <parent link= "$(arg namespace)/base_link" />
+        <child link= "depth_camera_link" />
+        <!-- <origin xyz= "0.55 0 3 " rpy= "0 0 0"/> -->
+        <origin xyz="-0.8 0 1.02" rpy="0 0 3.14159"/>
+    </joint>
+  <!-- optical link and joint for rviz -->
+  <link name= "depth_camera_optical_link"></link>
+  <joint name= "depth_camera_optical_joint" type= "fixed">
+      <parent link= "depth_camera_link" />
+      <child link= "depth_camera_optical_link" />
+      <origin xyz= "0 0 0 " rpy= "-1.57 0 -1.57"/>
+  </joint>
+  <gazebo reference= "depth_camera_link">
+      <material>Gazebo/Red</material>
+      <sensor name= "depth_camera_link" type= "depth">
+          <visualize>true</visualize>
+          <updateRate>10</updateRate>
+          <camera>
+              <horizontal_fov>1.57</horizontal_fov>
+              <vertical_fov>0.698</vertical_fov>
+              <image>
+                  <width>160</width>
+                  <height>100</height>
+              </image>
+              <clip>
+                  <near>0.1</near>
+                  <far>5.0</far>
+              </clip>
+          </camera>
+          <plugin name="depth_camera_sensor" filename="libgazebo_ros_openni_kinect.so">
+              <cameraName>depth_camera</cameraName>
+              <frameName>$(arg namespace)/depth_camera_optical_link</frameName>
+              <alwaysOn>true</alwaysOn>
+              <pointCloudTopicName>points</pointCloudTopicName>
+              <imageTopicName>rgb/image_raw</imageTopicName>
+              <depthImageTopicName>depth/image_raw</depthImageTopicName>
+              <cameraInfoTopicName>rgb/camera_info</cameraInfoTopicName>
+              <depthImageCameraInfoTopicName>depth/camera_info</depthImageCameraInfoTopicName>
+              <!-- <baseline>0.1</baseline> -->
+          </plugin>
+      </sensor>
+  </gazebo>
   <!-- imu sensor -->
   <link name= "imu_link">
@@ -155,15 +232,3 @@
     </sensor>
   </gazebo>
-  <xacro:default_joint_state_publisher namespace="$(arg namespace)" update_rate="50"/>
-  <!-- Initilizing thruster macro, might use another macro to achieve thrusters -->
-  <xacro:thruster_macro namespace="$(arg namespace)" thruster_id="0" mesh_scale="1">
-    <origin xyz="0.6650895 0.367385 0.828822" rpy="0 0 ${3*pi/4}"/>
-  </xacro:thruster_macro>
-  <xacro:thruster_macro namespace="$(arg namespace)" thruster_id="1" mesh_scale="1">
-    <origin xyz="0.665895 -0.367385 0.828822" rpy="0 0 ${-3*pi/4}"/>
-  </xacro:thruster_macro>
-  <!-- initilizing Sonar macro -->
-  <xacro:forward_multibeam_sonar_m450_130 namespace="$(arg namespace)" parent_link="$(arg namespace)/base_link" visualize="$(arg visualize)">
-    <origin xyz="-0.9 0 0.97" rpy="0 0 3.14159"/>
-  </xacro:forward_multibeam_sonar_m450_130>
 </robot>

File: urdf/tms_second_nouse.xacro (robot description, xacro)
@@ -3,10 +3,9 @@
   <!-- Necessary for sonar to work -->
   <xacro:arg name="namespace" default="tms"/>
-  <xacro:arg name="visualize" default="true"/>
-  <xacro:include filename="$(find deep_ocean)/urdf/sonar_snippets.xacro" />
+  <!-- <xacro:include filename="$(find uuv_sensor_ros_plugins)/urdf/sonar_snippets.xacro" /> -->
   <!-- Necessary for thruster_macro to work -->
   <xacro:include filename="$(find deep_ocean)/urdf/actuators.xacro" />
   <xacro:include filename="$(find uuv_descriptions)/urdf/common.urdf.xacro" />
-  <xacro:include filename="$(find deep_ocean)/urdf/thruster_snippets.xacro" />
+  <xacro:include filename="$(find uuv_gazebo_ros_plugins)/urdf/thruster_snippets.xacro" />
   <!-- Necessary for state publishing -->
   <xacro:include filename="$(find uuv_gazebo_ros_plugins)/urdf/misc.xacro" />
@@ -14,5 +13,5 @@
   <xacro:property name="fluid_density" value="1028"/>
   <!-- Scaling Factor for the TMS. Greater size means it's easier to dock -->
-  <xacro:property name="scale_factor" value="1"/> <!-- Change this to scale up/down -->
+  <xacro:property name="scale_factor" value="1.0"/> <!-- Change this to scale up/down -->
   <!-- Original Dimensions of the TMS -->
   <xacro:property name="size_x_orig" value="1.64"/>
@@ -24,9 +23,9 @@
   <xacro:property name="size_z" value="${size_z_orig * scale_factor}"/>
   <!-- Mass (Scaled) -->
-  <xacro:property name="mass" value="${550 * (scale_factor * scale_factor * scale_factor)}"/>
+  <xacro:property name="mass" value="${550.0 * (scale_factor * scale_factor * scale_factor)}"/>
   <!-- Volume (to ensure neutral buoyancy) -->
   <xacro:property name="volume" value="${mass / fluid_density}"/>
   <!-- Center of Buoyancy (adjusted based on height) -->
-  <xacro:property name="cob_z" value="${0.6 * size_z}"/>
+  <xacro:property name="cob_z" value="${0.5 * size_z}"/>
   <!-- Inertia Calculation -->
   <xacro:property name="ixx" value="${(1/12) * mass * (size_y * size_y + size_z * size_z)}"/>
@@ -54,18 +53,16 @@
     </collision>
   </link>
-  <!-- Spawning in ArUco marker -->
-  <link name="$(arg namespace)/aruco_marker">
-  <visual>
-    <origin xyz="0.25 0 0.2" rpy="0 0 0"/>  <!-- Adjust position as needed -->
-    <geometry>
-      <mesh filename="file://$(find deep_ocean)/meshes/Marker0.dae"/>
-    </geometry>
-  </visual>
-  </link>
-  <joint name="$(arg namespace)/aruco_joint" type="fixed">
-    <parent link="$(arg namespace)/base_link"/>  <!-- Adjust parent as needed -->
-    <child link="$(arg namespace)/aruco_marker"/>
-    <origin xyz="0 0 0" rpy="0 0 0"/>  <!-- Position on top front of vehicle -->
+  <!-- An attempt to restrict movement in z axis -->
+  <!--joint name="xy_plane_joint" type="planar">
+    <parent link="world"/>
+    <child link="base_link"/>
+    <axis xyz="1 0 0"/>
+    <axis2 xyz="0 1 0"/>
   </joint>
+  <joint name="yaw_joint" type="continuous">
+    <parent link="world"/>
+    <child link="base_link"/>
+    <axis xyz="0 0 1"/>
+  </joint-->
   <gazebo>
     <plugin name="uuv_plugin" filename="libuuv_underwater_object_ros_plugin.so">
@@ -74,5 +71,5 @@
       <debug>0</debug>
       <link name="$(arg namespace)/base_link">
-        <neutrally_buoyant>1</neutrally_buoyant>  <!-- Ensures mass and volume decide float/sink -->
+        <neutrally_buoyant>0</neutrally_buoyant>  <!-- Ensures mass and volume decide float/sink -->
         <volume>${volume}</volume>
         <box>
@@ -107,4 +104,82 @@
     </plugin>
   </gazebo>
+  <xacro:default_joint_state_publisher namespace="$(arg namespace)" update_rate="50"/>
+  <!-- Initilizing thruster macro, might use another macro to achieve thrusters -->
+  <xacro:thruster_macro namespace="$(arg namespace)" thruster_id="0">
+    <origin xyz="0.6650895 0.367385 0.828822" rpy="0 0 ${3*pi/4}"/>
+  </xacro:thruster_macro>
+  <xacro:thruster_macro namespace="$(arg namespace)" thruster_id="1">
+    <origin xyz="0.665895 -0.367385 0.828822" rpy="0 0 ${-3*pi/4}"/>
+  </xacro:thruster_macro>
+  <!-- initilizing Sonar macro -->
+  <!-- bruker denne som referanse til hjemmebygd sonar -->
+  <!-- <xacro:forward_multibeam_sonar_m450_130 namespace="$(arg namespace)" parent_link="$(arg namespace)/base_link">
+    <origin xyz="-0.9 0 1.02" rpy="0 0 3.14159"/>
+  </xacro:forward_multibeam_sonar_m450_130> -->
+<!-- kanskje prøve å etterligne denne https://waterlinked.com/shop/wl-21045-2-sonar-3d-15-689 -->
+  <link name= "depth_camera_link">
+      <visual>
+          <geometry>
+              <box size= "0.04 0.12 0.08" />
+          </geometry>
+          <material name= "red" >
+              <color rgba= "1 0 0 1" />
+          </material>
+      </visual>
+      <inertial>
+          <!-- <mass value= "0.39" /> -->
+          <mass value= "0.0" />
+          <origin xyz= "0 0 0" />
+          <inertia ixx= "0.1" ixy= "0.0" ixz= "0.0" iyy= "0.1" iyz= "0.0" izz= "0.1" />
+      </inertial>
+      <collision>
+          <geometry>
+              <box size= "0.04 0.12 0.08" />
+          </geometry>
+      </collision>
+  </link>
+    <joint name= "depth_camera_joint" type= "fixed">
+        <parent link= "$(arg namespace)/base_link" />
+        <child link= "depth_camera_link" />
+        <!-- <origin xyz= "0.55 0 3 " rpy= "0 0 0"/> -->
+        <origin xyz="-0.8 0 1.02" rpy="0 0 3.14159"/>
+    </joint>
+  <!-- optical link and joint for rviz -->
+  <link name= "depth_camera_optical_link"></link>
+  <joint name= "depth_camera_optical_joint" type= "fixed">
+      <parent link= "depth_camera_link" />
+      <child link= "depth_camera_optical_link" />
+      <origin xyz= "0 0 0 " rpy= "-1.57 0 -1.57"/>
+  </joint>
+  <gazebo reference= "depth_camera_link">
+      <material>Gazebo/Red</material>
+      <sensor name= "depth_camera_link" type= "depth">
+          <visualize>true</visualize>
+          <updateRate>10</updateRate>
+          <camera>
+              <horizontal_fov>1.57</horizontal_fov>
+              <vertical_fov>0.698</vertical_fov>
+              <image>
+                  <width>160</width>
+                  <height>100</height>
+              </image>
+              <clip>
+                  <near>0.1</near>
+                  <far>5.0</far>
+              </clip>
+          </camera>
+          <plugin name="depth_camera_sensor" filename="libgazebo_ros_openni_kinect.so">
+              <cameraName>depth_camera</cameraName>
+              <frameName>$(arg namespace)/depth_camera_optical_link</frameName>
+              <alwaysOn>true</alwaysOn>
+              <pointCloudTopicName>points</pointCloudTopicName>
+              <imageTopicName>rgb/image_raw</imageTopicName>
+              <depthImageTopicName>depth/image_raw</depthImageTopicName>
+              <cameraInfoTopicName>rgb/camera_info</cameraInfoTopicName>
+              <depthImageCameraInfoTopicName>depth/camera_info</depthImageCameraInfoTopicName>
+              <!-- <baseline>0.1</baseline> -->
+          </plugin>
+      </sensor>
+  </gazebo>
   <!-- imu sensor -->
   <link name= "imu_link">
@@ -155,15 +230,3 @@
     </sensor>
   </gazebo>
-  <xacro:default_joint_state_publisher namespace="$(arg namespace)" update_rate="50"/>
-  <!-- Initilizing thruster macro, might use another macro to achieve thrusters -->
-  <xacro:thruster_macro namespace="$(arg namespace)" thruster_id="0" mesh_scale="1">
-    <origin xyz="0.6650895 0.367385 0.828822" rpy="0 0 ${3*pi/4}"/>
-  </xacro:thruster_macro>
-  <xacro:thruster_macro namespace="$(arg namespace)" thruster_id="1" mesh_scale="1">
-    <origin xyz="0.665895 -0.367385 0.828822" rpy="0 0 ${-3*pi/4}"/>
-  </xacro:thruster_macro>
-  <!-- initilizing Sonar macro -->
-  <xacro:forward_multibeam_sonar_m450_130 namespace="$(arg namespace)" parent_link="$(arg namespace)/base_link" visualize="$(arg visualize)">
-    <origin xyz="-0.9 0 0.97" rpy="0 0 3.14159"/>
-  </xacro:forward_multibeam_sonar_m450_130>
 </robot>
