Commit message: Add files via upload

File: urdf/rov.xacro (robot description, xacro)
@@ -119,3 +119,51 @@
         </plugin>
     </gazebo>
+  <!-- imu sensor -->
+  <link name= "imu_link">
+      <visual>
+          <geometry>
+              <box size= "0.01 0.01 0.01" />
+          </geometry>
+          <material name= "red" >
+              <color rgba= "1 0 0 1" />
+          </material>
+      </visual>
+      <inertial>
+          <!-- <mass value= "0.39" /> -->
+          <mass value= "0.0" />
+          <origin xyz= "0 0 0" />
+          <inertia ixx= "0.1" ixy= "0.0" ixz= "0.0" iyy= "0.1" iyz= "0.0" izz= "0.1" />
+      </inertial>
+      <collision>
+          <geometry>
+              <box size= "0.01 0.01 0.01" />
+          </geometry>
+      </collision>
+  </link>
+  <joint name= "imu_joint" type= "fixed">
+      <parent link= "$(arg namespace)/base_link" />
+      <child link= "imu_link" />
+      <!-- <origin xyz= "0.55 0 3 " rpy= "0 0 0"/> -->
+      <origin xyz="0 0 0.81" rpy="0 0 0"/>
+  </joint>
+  <gazebo reference="imu_link">
+    <gravity>true</gravity>
+    <sensor name="imu_sensor" type="imu">
+      <always_on>true</always_on>
+      <update_rate>10</update_rate>
+      <visualize>true</visualize>
+      <topic>__default_topic__</topic>
+      <plugin filename="libgazebo_ros_imu_sensor.so" name="imu_plugin">
+        <topicName>imu</topicName>
+        <bodyName>imu_link</bodyName>
+        <updateRateHZ>10.0</updateRateHZ>
+        <gaussianNoise>0.0</gaussianNoise>
+        <xyzOffset>0 0 0</xyzOffset>
+        <rpyOffset>0 0 0</rpyOffset>
+        <frameName>imu_link</frameName>
+        <initialOrientationAsReference>false</initialOrientationAsReference>
+      </plugin>
+      <pose>0 0 0 0 0 0</pose>
+    </sensor>
+  </gazebo>
 </robot>

File: urdf/tms.xacro (robot description, xacro)
@@ -54,18 +54,4 @@
     </collision>
   </link>
-  <!-- Spawning in ArUco marker -->
-  <link name="$(arg namespace)/aruco_marker">
-  <visual>
-    <origin xyz="0.25 0 0.2" rpy="0 0 0"/>  <!-- Adjust position as needed -->
-    <geometry>
-      <mesh filename="file://$(find deep_ocean)/meshes/Marker0.dae"/>
-    </geometry>
-  </visual>
-  </link>
-  <joint name="$(arg namespace)/aruco_joint" type="fixed">
-    <parent link="$(arg namespace)/base_link"/>  <!-- Adjust parent as needed -->
-    <child link="$(arg namespace)/aruco_marker"/>
-    <origin xyz="0 0 0" rpy="0 0 0"/>  <!-- Position on top front of vehicle -->
-  </joint>
   <gazebo>
     <plugin name="uuv_plugin" filename="libuuv_underwater_object_ros_plugin.so">
@@ -165,5 +151,19 @@
   <!-- initilizing Sonar macro -->
   <xacro:forward_multibeam_sonar_m450_130 namespace="$(arg namespace)" parent_link="$(arg namespace)/base_link" visualize="$(arg visualize)">
-    <origin xyz="-0.9 0 0.97" rpy="0 0 3.14159"/>
+    <origin xyz="-0.9 0 0.97" rpy="0 0.13 3.14159"/>
   </xacro:forward_multibeam_sonar_m450_130>
+  <!-- Spawning in ArUco marker -->
+  <link name="$(arg namespace)/aruco_marker">
+  <visual>
+    <origin xyz="0.25 0 0.41" rpy="${pi/2} 0 ${-pi/2}"/>
+    <geometry>
+      <mesh filename="file://$(find deep_ocean)/materials/textures/marker_0.dae" scale="0.6 0.6 0.6"/>
+    </geometry>
+  </visual>
+  </link>
+  <joint name="$(arg namespace)/aruco_joint" type="fixed">
+    <parent link="$(arg namespace)/base_link"/>
+    <child link="$(arg namespace)/aruco_marker"/>
+    <origin xyz="0 0 0" rpy="0 0 0"/>
+  </joint>
 </robot>

File: urdf/tms_second.xacro (robot description, xacro)
@@ -54,18 +54,4 @@
     </collision>
   </link>
-  <!-- Spawning in ArUco marker -->
-  <link name="$(arg namespace)/aruco_marker">
-  <visual>
-    <origin xyz="0.25 0 0.2" rpy="0 0 0"/>  <!-- Adjust position as needed -->
-    <geometry>
-      <mesh filename="file://$(find deep_ocean)/meshes/Marker0.dae"/>
-    </geometry>
-  </visual>
-  </link>
-  <joint name="$(arg namespace)/aruco_joint" type="fixed">
-    <parent link="$(arg namespace)/base_link"/>  <!-- Adjust parent as needed -->
-    <child link="$(arg namespace)/aruco_marker"/>
-    <origin xyz="0 0 0" rpy="0 0 0"/>  <!-- Position on top front of vehicle -->
-  </joint>
   <gazebo>
     <plugin name="uuv_plugin" filename="libuuv_underwater_object_ros_plugin.so">
@@ -232,3 +218,31 @@
     </sensor>
   </gazebo>
+  <!-- Spawning in ArUco marker -->
+  <link name="$(arg namespace)/aruco_marker">
+  <visual>
+    <origin xyz="0.25 0 0.41" rpy="${pi/2} 0 ${-pi/2}"/>
+    <geometry>
+      <mesh filename="file://$(find deep_ocean)/materials/textures/marker_0.dae" scale="0.6 0.6 0.6"/>
+    </geometry>
+  </visual>
+  </link>
+  <joint name="$(arg namespace)/aruco_joint" type="fixed">
+    <parent link="$(arg namespace)/base_link"/>
+    <child link="$(arg namespace)/aruco_marker"/>
+    <origin xyz="0 0 0" rpy="0 0 0"/>
+  </joint>
+  <!-- Spawning a calibration board of 7x10 dimension -->
+  <link name="$(arg namespace)/calibration_board">
+  <visual>
+    <origin xyz="-2 1 0.4" rpy="${pi/2} 0 ${-pi/2}"/>
+    <geometry>
+      <mesh filename="file://$(find deep_ocean)/materials/textures/checkerboard_7x10_bordered.dae" scale="0.6 0.6 0.6"/>
+    </geometry>
+  </visual>
+  </link>
+  <joint name="$(arg namespace)/checker_joint" type="fixed">
+    <parent link="$(arg namespace)/base_link"/>
+    <child link="$(arg namespace)/calibration_board"/>
+    <origin xyz="0 0 0" rpy="0 0 0"/>
+  </joint>
 </robot>

Commit message: Add files via upload

File: urdf/rov.xacro (robot description, xacro)
@@ -167,3 +167,63 @@
     </sensor>
   </gazebo>
+      <!-- camera -->
+    <link name= "camera_link">
+        <visual>
+            <geometry>
+                <box size= "0.1 0.1 0.1" />
+            </geometry>
+            <material name= "red" >
+                <color rgba= "1 0 0 1" />
+            </material>
+        </visual>
+        <inertial>
+            <mass value= "0.2" />
+            <origin xyz= "0 0 0" />
+            <inertia ixx= "0.1" ixy= "0.0" ixz= "0.0" iyy= "0.1" iyz= "0.0" izz= "0.1" />
+        </inertial>
+        <collision>
+            <geometry>
+                <box size= "0.1 0.1 0.1" />
+            </geometry>
+        </collision>
+    </link>
+    <joint name= "camera_joint" type= "fixed">
+        <parent link= "$(arg namespace)/base_link" />
+        <child link= "camera_link" />
+        <origin xyz="0.63 0 0.4" rpy="0 0 0"/>
+    </joint>
+    <link name= "camera_link_optical"></link>
+    <joint name= "camera_optical_joint" type= "fixed">
+        <parent link= "camera_link" />
+        <child link= "camera_link_optical" />
+        <origin xyz= "0 0 0 " rpy= "-1.57 0 -1.57"/>
+    </joint>
+    <gazebo reference= "camera_link">
+        <material>Gazebo/Red</material>
+        <sensor type= "camera" name= "camera_sensor">
+            <pose>0 0 0 0 0 0</pose>
+            <visualize>true</visualize>
+            <update_rate>30</update_rate>
+            <camera>
+                <horizontal_fov>1.047</horizontal_fov>
+                <image>
+                    <width>640</width>
+                    <height>480</height>
+                    <format>R8G8B8</format>
+                </image>
+                <clip>
+                    <near>0.1</near>
+                    <far>10</far>
+                </clip>
+            </camera>
+            <plugin name= "camera_controller" filename= "libgazebo_ros_camera.so" >
+                <frameName>camera_link_optical</frameName>
+                <alwaysOn>true</alwaysOn>
+                <updateRate>0.0</updateRate>
+                <cameraName>camera</cameraName>
+                <imageTopicName>image_raw</imageTopicName>
+                <cameraInfoTopicName>camera_info</cameraInfoTopicName>
+            </plugin>
+        </sensor>
+    </gazebo>
 </robot>
