Commit message: Add files via upload

File: robots/tms_2d_sonar.xacro (robot description, xacro)
@@ -3,8 +3,10 @@
   <!-- Necessary for sonar to work -->
   <xacro:arg name="namespace" default="tms"/>
+  <xacro:arg name="visualize" default="true"/>
+  <xacro:include filename="$(find deep_ocean)/urdf/sonar_snippets.xacro" />
   <!-- Necessary for thruster_macro to work -->
   <xacro:include filename="$(find deep_ocean)/urdf/actuators.xacro" />
   <xacro:include filename="$(find uuv_descriptions)/urdf/common.urdf.xacro" />
-  <xacro:include filename="$(find uuv_gazebo_ros_plugins)/urdf/thruster_snippets.xacro" />
+  <xacro:include filename="$(find deep_ocean)/urdf/thruster_snippets.xacro" />
   <!-- Necessary for state publishing -->
   <xacro:include filename="$(find uuv_gazebo_ros_plugins)/urdf/misc.xacro" />
@@ -12,5 +14,5 @@
   <xacro:property name="fluid_density" value="1028"/>
   <!-- Scaling Factor for the TMS. Greater size means it's easier to dock -->
-  <xacro:property name="scale_factor" value="1.0"/> <!-- Change this to scale up/down -->
+  <xacro:property name="scale_factor" value="1"/> <!-- Change this to scale up/down -->
   <!-- Original Dimensions of the TMS -->
   <xacro:property name="size_x_orig" value="1.64"/>
@@ -22,9 +24,9 @@
   <xacro:property name="size_z" value="${size_z_orig * scale_factor}"/>
   <!-- Mass (Scaled) -->
-  <xacro:property name="mass" value="${550.0 * (scale_factor * scale_factor * scale_factor)}"/>
+  <xacro:property name="mass" value="${550 * (scale_factor * scale_factor * scale_factor)}"/>
   <!-- Volume (to ensure neutral buoyancy) -->
   <xacro:property name="volume" value="${mass / fluid_density}"/>
   <!-- Center of Buoyancy (adjusted based on height) -->
-  <xacro:property name="cob_z" value="${0.5 * size_z}"/>
+  <xacro:property name="cob_z" value="${0.6 * size_z}"/>
   <!-- Inertia Calculation -->
   <xacro:property name="ixx" value="${(1/12) * mass * (size_y * size_y + size_z * size_z)}"/>
@@ -52,16 +54,4 @@
     </collision>
   </link>
-  <!-- An attempt to restrict movement in z axis -->
-  <!--joint name="xy_plane_joint" type="planar">
-    <parent link="world"/>
-    <child link="base_link"/>
-    <axis xyz="1 0 0"/>
-    <axis2 xyz="0 1 0"/>
-  </joint>
-  <joint name="yaw_joint" type="continuous">
-    <parent link="world"/>
-    <child link="base_link"/>
-    <axis xyz="0 0 1"/>
-  </joint-->
   <gazebo>
     <plugin name="uuv_plugin" filename="libuuv_underwater_object_ros_plugin.so">
@@ -70,5 +60,5 @@
       <debug>0</debug>
       <link name="$(arg namespace)/base_link">
-        <neutrally_buoyant>0</neutrally_buoyant>  <!-- Ensures mass and volume decide float/sink -->
+        <neutrally_buoyant>1</neutrally_buoyant>  <!-- Ensures mass and volume decide float/sink -->
         <volume>${volume}</volume>
         <box>
@@ -102,82 +92,4 @@
       </link>
     </plugin>
-  </gazebo>
-  <xacro:default_joint_state_publisher namespace="$(arg namespace)" update_rate="50"/>
-  <!-- Initilizing thruster macro, might use another macro to achieve thrusters -->
-  <xacro:thruster_macro namespace="$(arg namespace)" thruster_id="0">
-    <origin xyz="0.6650895 0.367385 0.828822" rpy="0 0 ${3*pi/4}"/>
-  </xacro:thruster_macro>
-  <xacro:thruster_macro namespace="$(arg namespace)" thruster_id="1">
-    <origin xyz="0.665895 -0.367385 0.828822" rpy="0 0 ${-3*pi/4}"/>
-  </xacro:thruster_macro>
-  <!-- initilizing Sonar macro -->
-  <!-- bruker denne som referanse til hjemmebygd sonar -->
-  <!-- <xacro:forward_multibeam_sonar_m450_130 namespace="$(arg namespace)" parent_link="$(arg namespace)/base_link">
-    <origin xyz="-0.9 0 1.02" rpy="0 0 3.14159"/>
-  </xacro:forward_multibeam_sonar_m450_130> -->
-<!-- kanskje prøve å etterligne denne https://waterlinked.com/shop/wl-21045-2-sonar-3d-15-689 -->
-  <link name= "depth_camera_link">
-      <visual>
-          <geometry>
-              <box size= "0.04 0.12 0.08" />
-          </geometry>
-          <material name= "red" >
-              <color rgba= "1 0 0 1" />
-          </material>
-      </visual>
-      <inertial>
-          <!-- <mass value= "0.39" /> -->
-          <mass value= "0.0" />
-          <origin xyz= "0 0 0" />
-          <inertia ixx= "0.1" ixy= "0.0" ixz= "0.0" iyy= "0.1" iyz= "0.0" izz= "0.1" />
-      </inertial>
-      <collision>
-          <geometry>
-              <box size= "0.04 0.12 0.08" />
-          </geometry>
-      </collision>
-  </link>
-    <joint name= "depth_camera_joint" type= "fixed">
-        <parent link= "$(arg namespace)/base_link" />
-        <child link= "depth_camera_link" />
-        <!-- <origin xyz= "0.55 0 3 " rpy= "0 0 0"/> -->
-        <origin xyz="-0.8 0 1.02" rpy="0 0 3.14159"/>
-    </joint>
-  <!-- optical link and joint for rviz -->
-  <link name= "depth_camera_optical_link"></link>
-  <joint name= "depth_camera_optical_joint" type= "fixed">
-      <parent link= "depth_camera_link" />
-      <child link= "depth_camera_optical_link" />
-      <origin xyz= "0 0 0 " rpy= "-1.57 0 -1.57"/>
-  </joint>
-  <gazebo reference= "depth_camera_link">
-      <material>Gazebo/Red</material>
-      <sensor name= "depth_camera_link" type= "depth">
-          <visualize>true</visualize>
-          <updateRate>10</updateRate>
-          <camera>
-              <horizontal_fov>1.57</horizontal_fov>
-              <vertical_fov>0.698</vertical_fov>
-              <image>
-                  <width>160</width>
-                  <height>100</height>
-              </image>
-              <clip>
-                  <near>0.1</near>
-                  <far>5.0</far>
-              </clip>
-          </camera>
-          <plugin name="depth_camera_sensor" filename="libgazebo_ros_openni_kinect.so">
-              <cameraName>depth_camera</cameraName>
-              <frameName>$(arg namespace)/depth_camera_optical_link</frameName>
-              <alwaysOn>true</alwaysOn>
-              <pointCloudTopicName>points</pointCloudTopicName>
-              <imageTopicName>rgb/image_raw</imageTopicName>
-              <depthImageTopicName>depth/image_raw</depthImageTopicName>
-              <cameraInfoTopicName>rgb/camera_info</cameraInfoTopicName>
-              <depthImageCameraInfoTopicName>depth/camera_info</depthImageCameraInfoTopicName>
-              <!-- <baseline>0.1</baseline> -->
-          </plugin>
-      </sensor>
   </gazebo>
   <!-- imu sensor -->
@@ -229,3 +141,29 @@
     </sensor>
   </gazebo>
+  <xacro:default_joint_state_publisher namespace="$(arg namespace)" update_rate="50"/>
+  <!-- Initilizing thruster macro, might use another macro to achieve thrusters -->
+  <xacro:thruster_macro namespace="$(arg namespace)" thruster_id="0" mesh_scale="1">
+    <origin xyz="0.6650895 0.367385 0.828822" rpy="0 0 ${3*pi/4}"/>
+  </xacro:thruster_macro>
+  <xacro:thruster_macro namespace="$(arg namespace)" thruster_id="1" mesh_scale="1">
+    <origin xyz="0.665895 -0.367385 0.828822" rpy="0 0 ${-3*pi/4}"/>
+  </xacro:thruster_macro>
+  <!-- initilizing Sonar macro -->
+  <xacro:forward_multibeam_sonar_m450_130 namespace="$(arg namespace)" parent_link="$(arg namespace)/base_link" visualize="$(arg visualize)">
+    <origin xyz="-0.9 0 0.97" rpy="0 0.13 3.14159"/>
+  </xacro:forward_multibeam_sonar_m450_130>
+  <!-- Spawning in ArUco 5x5 marker -->
+  <link name="$(arg namespace)/aruco_marker">
+  <visual>
+    <origin xyz="0.25 0 0.41" rpy="${pi/2} 0 ${-pi/2}"/>
+    <geometry>
+      <mesh filename="file://$(find deep_ocean)/materials/textures/marker_5x5_0.dae" scale="0.6 0.6 0.6"/>
+    </geometry>
+  </visual>
+  </link>
+  <joint name="$(arg namespace)/aruco_joint" type="fixed">
+    <parent link="$(arg namespace)/base_link"/>
+    <child link="$(arg namespace)/aruco_marker"/>
+    <origin xyz="0 0 0" rpy="0 0 0"/>
+  </joint>
 </robot>

File: robots/tms_3d_sonar.xacro (robot description, xacro)
@@ -3,8 +3,10 @@
   <!-- Necessary for sonar to work -->
   <xacro:arg name="namespace" default="tms"/>
+  <xacro:arg name="visualize" default="true"/>
+  <xacro:include filename="$(find deep_ocean)/urdf/sonar_snippets.xacro" />
   <!-- Necessary for thruster_macro to work -->
   <xacro:include filename="$(find deep_ocean)/urdf/actuators.xacro" />
   <xacro:include filename="$(find uuv_descriptions)/urdf/common.urdf.xacro" />
-  <xacro:include filename="$(find uuv_gazebo_ros_plugins)/urdf/thruster_snippets.xacro" />
+  <xacro:include filename="$(find deep_ocean)/urdf/thruster_snippets.xacro" />
   <!-- Necessary for state publishing -->
   <xacro:include filename="$(find uuv_gazebo_ros_plugins)/urdf/misc.xacro" />
@@ -12,5 +14,5 @@
   <xacro:property name="fluid_density" value="1028"/>
   <!-- Scaling Factor for the TMS. Greater size means it's easier to dock -->
-  <xacro:property name="scale_factor" value="1.0"/> <!-- Change this to scale up/down -->
+  <xacro:property name="scale_factor" value="1"/> <!-- Change this to scale up/down -->
   <!-- Original Dimensions of the TMS -->
   <xacro:property name="size_x_orig" value="1.64"/>
@@ -22,9 +24,9 @@
   <xacro:property name="size_z" value="${size_z_orig * scale_factor}"/>
   <!-- Mass (Scaled) -->
-  <xacro:property name="mass" value="${550.0 * (scale_factor * scale_factor * scale_factor)}"/>
+  <xacro:property name="mass" value="${550 * (scale_factor * scale_factor * scale_factor)}"/>
   <!-- Volume (to ensure neutral buoyancy) -->
   <xacro:property name="volume" value="${mass / fluid_density}"/>
   <!-- Center of Buoyancy (adjusted based on height) -->
-  <xacro:property name="cob_z" value="${0.5 * size_z}"/>
+  <xacro:property name="cob_z" value="${0.6 * size_z}"/>
   <!-- Inertia Calculation -->
   <xacro:property name="ixx" value="${(1/12) * mass * (size_y * size_y + size_z * size_z)}"/>
@@ -34,5 +36,5 @@
     <inertial>
       <mass value="${mass}"/>
-      <origin xyz="0 0 0" rpy="0 0 3.14159"/>
+      <origin xyz="0 0 0" rpy="0 0 3.14159"/>5
       <inertia ixx="${ixx}" ixy="0.0" ixz="0.0" iyy="${iyy}" iyz="0.0" izz="${izz}"/>
     </inertial>
@@ -52,16 +54,4 @@
     </collision>
   </link>
-  <!-- An attempt to restrict movement in z axis -->
-  <!--joint name="xy_plane_joint" type="planar">
-    <parent link="world"/>
-    <child link="base_link"/>
-    <axis xyz="1 0 0"/>
-    <axis2 xyz="0 1 0"/>
-  </joint>
-  <joint name="yaw_joint" type="continuous">
-    <parent link="world"/>
-    <child link="base_link"/>
-    <axis xyz="0 0 1"/>
-  </joint-->
   <gazebo>
     <plugin name="uuv_plugin" filename="libuuv_underwater_object_ros_plugin.so">
@@ -70,5 +60,5 @@
       <debug>0</debug>
       <link name="$(arg namespace)/base_link">
-        <neutrally_buoyant>0</neutrally_buoyant>  <!-- Ensures mass and volume decide float/sink -->
+        <neutrally_buoyant>1</neutrally_buoyant>  <!-- Ensures mass and volume decide float/sink -->
         <volume>${volume}</volume>
         <box>
@@ -105,80 +95,19 @@
   <xacro:default_joint_state_publisher namespace="$(arg namespace)" update_rate="50"/>
   <!-- Initilizing thruster macro, might use another macro to achieve thrusters -->
-  <xacro:thruster_macro namespace="$(arg namespace)" thruster_id="0">
+  <xacro:thruster_macro namespace="$(arg namespace)" thruster_id="0" mesh_scale="1">
     <origin xyz="0.6650895 0.367385 0.828822" rpy="0 0 ${3*pi/4}"/>
   </xacro:thruster_macro>
-  <xacro:thruster_macro namespace="$(arg namespace)" thruster_id="1">
+  <xacro:thruster_macro namespace="$(arg namespace)" thruster_id="1" mesh_scale="1">
     <origin xyz="0.665895 -0.367385 0.828822" rpy="0 0 ${-3*pi/4}"/>
   </xacro:thruster_macro>
   <!-- initilizing Sonar macro -->
-  <!-- bruker denne som referanse til hjemmebygd sonar -->
-  <!-- <xacro:forward_multibeam_sonar_m450_130 namespace="$(arg namespace)" parent_link="$(arg namespace)/base_link">
-    <origin xyz="-0.9 0 1.02" rpy="0 0 3.14159"/>
-  </xacro:forward_multibeam_sonar_m450_130> -->
+  <!--xacro:forward_multibeam_sonar_m450_130 namespace="$(arg namespace)" parent_link="$(arg namespace)/base_link" visualize="$(arg visualize)">
+    <origin xyz="-0.9 0 0.97" rpy="0 0 3.14159"/>
+  </xacro:forward_multibeam_sonar_m450_130-->
 <!-- kanskje prøve å etterligne denne https://waterlinked.com/shop/wl-21045-2-sonar-3d-15-689 -->
-  <link name= "depth_camera_link">
-      <visual>
-          <geometry>
-              <box size= "0.04 0.12 0.08" />
-          </geometry>
-          <material name= "red" >
-              <color rgba= "1 0 0 1" />
-          </material>
-      </visual>
-      <inertial>
-          <!-- <mass value= "0.39" /> -->
-          <mass value= "0.0" />
-          <origin xyz= "0 0 0" />
-          <inertia ixx= "0.1" ixy= "0.0" ixz= "0.0" iyy= "0.1" iyz= "0.0" izz= "0.1" />
-      </inertial>
-      <collision>
-          <geometry>
-              <box size= "0.04 0.12 0.08" />
-          </geometry>
-      </collision>
-  </link>
-    <joint name= "depth_camera_joint" type= "fixed">
-        <parent link= "$(arg namespace)/base_link" />
-        <child link= "depth_camera_link" />
-        <!-- <origin xyz= "0.55 0 3 " rpy= "0 0 0"/> -->
-        <origin xyz="-0.8 0 1.02" rpy="0 0 3.14159"/>
-    </joint>
-  <!-- optical link and joint for rviz -->
-  <link name= "depth_camera_optical_link"></link>
-  <joint name= "depth_camera_optical_joint" type= "fixed">
-      <parent link= "depth_camera_link" />
-      <child link= "depth_camera_optical_link" />
-      <origin xyz= "0 0 0 " rpy= "-1.57 0 -1.57"/>
-  </joint>
-  <gazebo reference= "depth_camera_link">
-      <material>Gazebo/Red</material>
-      <sensor name= "depth_camera_link" type= "depth">
-          <visualize>true</visualize>
-          <updateRate>10</updateRate>
-          <camera>
-              <horizontal_fov>1.57</horizontal_fov>
-              <vertical_fov>0.698</vertical_fov>
-              <image>
-                  <width>160</width>
-                  <height>100</height>
-              </image>
-              <clip>
-                  <near>0.1</near>
-                  <far>5.0</far>
-              </clip>
-          </camera>
-          <plugin name="depth_camera_sensor" filename="libgazebo_ros_openni_kinect.so">
-              <cameraName>depth_camera</cameraName>
-              <frameName>$(arg namespace)/depth_camera_optical_link</frameName>
-              <alwaysOn>true</alwaysOn>
-              <pointCloudTopicName>points</pointCloudTopicName>
-              <imageTopicName>rgb/image_raw</imageTopicName>
-              <depthImageTopicName>depth/image_raw</depthImageTopicName>
-              <cameraInfoTopicName>rgb/camera_info</cameraInfoTopicName>
-              <depthImageCameraInfoTopicName>depth/camera_info</depthImageCameraInfoTopicName>
-              <!-- <baseline>0.1</baseline> -->
-          </plugin>
-      </sensor>
-  </gazebo>
+  <xacro:sonar_3d
+    parent_link="$(arg namespace)/base_link"
+    namespace="$(arg namespace)"
+    visualize="$(arg visualize)"/>
   <!-- imu sensor -->
   <link name= "imu_link">
@@ -229,3 +158,31 @@
     </sensor>
   </gazebo>
+  <!-- Spawning in ArUco 5x5 marker -->
+  <link name="$(arg namespace)/aruco_marker">
+  <visual>
+    <origin xyz="0.25 0 0.41" rpy="${pi/2} 0 ${-pi/2}"/>
+    <geometry>
+      <mesh filename="file://$(find deep_ocean)/materials/textures/marker_5x5_0.dae" scale="0.6 0.6 0.6"/>
+    </geometry>
+  </visual>
+  </link>
+  <joint name="$(arg namespace)/aruco_joint" type="fixed">
+    <parent link="$(arg namespace)/base_link"/>
+    <child link="$(arg namespace)/aruco_marker"/>
+    <origin xyz="0 0 0" rpy="0 0 0"/>
+  </joint>
+  <!-- Spawning a calibration board of 7x10 dimension -->
+  <!-- <link name="$(arg namespace)/calibration_board">
+  <visual>
+    <origin xyz="-2 1 0.4" rpy="${pi/2} 0 ${-pi/2}"/>
+    <geometry>
+      <mesh filename="file://$(find deep_ocean)/materials/textures/checkerboard_7x10_bordered.dae" scale="0.6 0.6 0.6"/>
+    </geometry>
+  </visual>
+  </link>
+  <joint name="$(arg namespace)/checker_joint" type="fixed">
+    <parent link="$(arg namespace)/base_link"/>
+    <child link="$(arg namespace)/calibration_board"/>
+    <origin xyz="0 0 0" rpy="0 0 0"/>
+  </joint> -->
 </robot>

File: urdf/sonar_snippets.xacro (robot description, xacro)
@@ -21,29 +21,4 @@
       <origin xyz="0 0 0" rpy="0 ${0.5*pi} 0"/>
     </collision>
-  </xacro:macro>
-  <!-- Side scan sonar -->
-  <xacro:macro name="sidescan_sonar" params="namespace parent_link suffix *origin">
-    <xacro:multibeam_sonar
-      namespace="${namespace}"
-      suffix="${suffix}"
-      parent_link="${parent_link}"
-      topic="sss_${suffix}"
-      mass="0.015"
-      update_rate="2"
-      samples="60"
-      fov="${pi/3.0}"
-      range_min="1.0"
-      range_max="200.0"
-      range_stddev="0.027"
-      mesh="">
-      <inertia ixx="0.00001" ixy="0.0" ixz="0.0" iyy="0.00001" iyz="0.0" izz="0.00001" />
-      <xacro:insert_block name="origin" />
-      <visual>
-        <origin xyz="0 0 0" rpy="0 0 0"/>
-        <geometry>
-          <box size="0.001 0.001 0.001"/>
-        </geometry>
-      </visual>
-    </xacro:multibeam_sonar>
   </xacro:macro>
   <!-- Inspired by m450-130: http://www.blueview.com/products/2d-imaging-sonar/m900-series/ -->
@@ -153,20 +128,68 @@
   </gazebo>
   </xacro:macro>
-<!-- This is a self defined sonar -->
-  <xacro:macro name="forward_looking_sonar_1" params="namespace parent_link *origin">
-    <xacro:forward_looking_sonar
-      namespace="${namespace}"
-      suffix=""
-      parent_link="${parent_link}"
-      topic="sonar"
-      mass="0.015"
-      update_rate="25"
-      samples="768"
-      fov="2.27"
-      width="5"
-      height="5">
-      <inertia ixx="0.00001" ixy="0.0" ixz="0.0" iyy="0.00001" iyz="0.0" izz="0.00001" />
-      <xacro:insert_block name="origin" />
-    </xacro:forward_looking_sonar>
+  <!-- Macro a 3d depth sonar -->
+  <xacro:macro name="sonar_3d" params="parent_link namespace visualize:=true">
+    <link name="${namespace}/sonar_3d_link">
+      <visual>
+        <geometry>
+          <box size="0.04 0.12 0.08"/>
+        </geometry>
+        <material name="red">
+          <color rgba="1 0 0 1"/>
+        </material>
+      </visual>
+      <inertial>
+        <mass value="0.0"/>
+        <origin xyz="0 0 0"/>
+        <inertia ixx="0.1" ixy="0.0" ixz="0.0" iyy="0.1" iyz="0.0" izz="0.1"/>
+      </inertial>
+      <collision>
+        <geometry>
+          <box size="0.04 0.12 0.08"/>
+        </geometry>
+      </collision>
+    </link>
+    <joint name="${namespace}/sonar_3d_joint" type="fixed">
+      <parent link="${parent_link}"/>
+      <child link="${namespace}/sonar_3d_link"/>
+      <origin xyz="-0.8 0 1.02" rpy="0 0 3.14159"/>
+    </joint>
+    <link name="${namespace}/sonar_3d_optical_link"/>
+    <joint name="${namespace}/sonar_3d_optical_joint" type="fixed">
+      <parent link="${namespace}/sonar_3d_link"/>
+      <child link="${namespace}/sonar_3d_optical_link"/>
+      <origin xyz="0 0 0" rpy="-1.57 0 -1.57"/>
+    </joint>
+    <xacro:if value="${visualize}">
+      <gazebo reference="${namespace}/sonar_3d_link">
+        <material>Gazebo/Red</material>
+        <sensor name="sonar_3d_sensor" type="depth">
+          <visualize>true</visualize>
+          <updateRate>10</updateRate>
+          <camera>
+            <horizontal_fov>1.57</horizontal_fov>
+            <vertical_fov>0.698</vertical_fov>
+            <image>
+              <width>160</width>
+              <height>100</height>
+            </image>
+            <clip>
+              <near>0.1</near>
+              <far>5.0</far>
+            </clip>
+          </camera>
+          <plugin name="sonar_3d_plugin" filename="libgazebo_ros_openni_kinect.so">
+            <cameraName>${namespace}/sonar_3d</cameraName>
+            <frameName>${namespace}/sonar_3d_optical_link</frameName>
+            <alwaysOn>true</alwaysOn>
+            <pointCloudTopicName>points</pointCloudTopicName>
+            <imageTopicName>rgb/image_raw</imageTopicName>
+            <depthImageTopicName>depth/image_raw</depthImageTopicName>
+            <cameraInfoTopicName>rgb/camera_info</cameraInfoTopicName>
+            <depthImageCameraInfoTopicName>depth/camera_info</depthImageCameraInfoTopicName>
+          </plugin>
+        </sensor>
+      </gazebo>
+    </xacro:if>
   </xacro:macro>
   <xacro:macro name="forward_looking_sonar"
