Commit message: Add files via upload

File: robots/tms_2d_sonar.xacro (robot description, xacro)
@@ -11,4 +11,6 @@
   <!-- Necessary for state publishing -->
   <xacro:include filename="$(find uuv_gazebo_ros_plugins)/urdf/misc.xacro" />
+  <!-- Necessary for ArUco markers and calibration bord -->
+  <xacro:include filename="$(find deep_ocean)/urdf/aruco_macro.xacro" />
   <!-- Fluid Density of Water (kg/m³) -->
   <xacro:property name="fluid_density" value="1028"/>
@@ -119,5 +121,5 @@
       <child link= "imu_link" />
       <!-- <origin xyz= "0.55 0 3 " rpy= "0 0 0"/> -->
-      <origin xyz="0 0 0.81" rpy="0 0 0"/>
+      <origin xyz="0 0 ${0.81*scale_factor}" rpy="0 0 0"/>
   </joint>
   <gazebo reference="imu_link">
@@ -143,27 +145,30 @@
   <xacro:default_joint_state_publisher namespace="$(arg namespace)" update_rate="50"/>
   <!-- Initilizing thruster macro, might use another macro to achieve thrusters -->
-  <xacro:thruster_macro namespace="$(arg namespace)" thruster_id="0" mesh_scale="1">
-    <origin xyz="0.6650895 0.367385 0.828822" rpy="0 0 ${3*pi/4}"/>
+  <xacro:thruster_macro namespace="$(arg namespace)" thruster_id="0" mesh_scale="${scale_factor}">
+    <origin xyz="${0.6650895*scale_factor} ${0.367385*scale_factor} ${0.828822*scale_factor}" rpy="0 0 ${3*pi/4}"/>
   </xacro:thruster_macro>
-  <xacro:thruster_macro namespace="$(arg namespace)" thruster_id="1" mesh_scale="1">
-    <origin xyz="0.665895 -0.367385 0.828822" rpy="0 0 ${-3*pi/4}"/>
+  <xacro:thruster_macro namespace="$(arg namespace)" thruster_id="1" mesh_scale="${scale_factor}">
+    <origin xyz="${0.665895*scale_factor} ${-0.367385*scale_factor} ${0.828822*scale_factor}" rpy="0 0 ${-3*pi/4}"/>
   </xacro:thruster_macro>
   <!-- initilizing Sonar macro -->
   <xacro:forward_multibeam_sonar_m450_130 namespace="$(arg namespace)" parent_link="$(arg namespace)/base_link" visualize="$(arg visualize)">
-    <origin xyz="-0.9 0 0.97" rpy="0 0.13 3.14159"/>
+    <origin xyz="${-0.9*scale_factor} 0 ${0.97*scale_factor}" rpy="0 0.13 3.14159"/>
   </xacro:forward_multibeam_sonar_m450_130>
-  <!-- Spawning in ArUco 5x5 marker -->
-  <link name="$(arg namespace)/aruco_marker">
-  <visual>
-    <origin xyz="0.25 0 0.41" rpy="${pi/2} 0 ${-pi/2}"/>
-    <geometry>
-      <mesh filename="file://$(find deep_ocean)/materials/textures/marker_5x5_0.dae" scale="0.6 0.6 0.6"/>
-    </geometry>
-  </visual>
-  </link>
-  <joint name="$(arg namespace)/aruco_joint" type="fixed">
-    <parent link="$(arg namespace)/base_link"/>
-    <child link="$(arg namespace)/aruco_marker"/>
-    <origin xyz="0 0 0" rpy="0 0 0"/>
-  </joint>
+    <!-- Spawning in ArUco 5x5 marker -->
+  <xacro:aruco_marker_5x5 namespace="$(arg namespace)" parent_link="$(arg namespace)/base_link" id="0" scale="${0.3*scale_factor}">
+    <origin xyz="${0.25*scale_factor} 0 ${0.66*scale_factor}" rpy="${pi/2} 0 ${-pi/2}"/>
+  </xacro:aruco_marker_5x5>
+    <!-- Spawning in ArUco 4x4 marker -->
+  <xacro:aruco_marker_4x4 namespace="$(arg namespace)" parent_link="$(arg namespace)/base_link" id="0" scale="${scale_factor}">
+    <origin xyz="${-0.8*scale_factor} ${0.5*scale_factor} ${0.97*scale_factor}" rpy="${pi/2} 0 ${-pi/2}"/>
+  </xacro:aruco_marker_4x4>
+  <xacro:aruco_marker_4x4 namespace="$(arg namespace)" parent_link="$(arg namespace)/base_link" id="1" scale="${scale_factor}">
+    <origin xyz="${-0.8*scale_factor} ${0.5*scale_factor} 0" rpy="${pi/2} 0 ${-pi/2}"/>
+  </xacro:aruco_marker_4x4>
+  <xacro:aruco_marker_4x4 namespace="$(arg namespace)" parent_link="$(arg namespace)/base_link" id="2" scale="${scale_factor}">
+    <origin xyz="${-0.8*scale_factor} ${-0.5*scale_factor} 0" rpy="${pi/2} 0 ${-pi/2}"/>
+  </xacro:aruco_marker_4x4>
+  <xacro:aruco_marker_4x4 namespace="$(arg namespace)" parent_link="$(arg namespace)/base_link" id="3" scale="${scale_factor}">
+    <origin xyz="${-0.8*scale_factor} ${-0.5*scale_factor} ${0.97*scale_factor}" rpy="${pi/2} 0 ${-pi/2}"/>
+  </xacro:aruco_marker_4x4>
 </robot>

File: robots/tms_3d_sonar.xacro (robot description, xacro)
@@ -11,8 +11,10 @@
   <!-- Necessary for state publishing -->
   <xacro:include filename="$(find uuv_gazebo_ros_plugins)/urdf/misc.xacro" />
+  <!-- Necessary for ArUco markers and calibration bord -->
+  <xacro:include filename="$(find deep_ocean)/urdf/aruco_macro.xacro" />
   <!-- Fluid Density of Water (kg/m³) -->
   <xacro:property name="fluid_density" value="1028"/>
   <!-- Scaling Factor for the TMS. Greater size means it's easier to dock -->
-  <xacro:property name="scale_factor" value="1"/> <!-- Change this to scale up/down -->
+  <xacro:property name="scale_factor" value="2"/> <!-- Change this to scale up/down -->
   <!-- Original Dimensions of the TMS -->
   <xacro:property name="size_x_orig" value="1.64"/>
@@ -94,20 +96,16 @@
   </gazebo>
   <xacro:default_joint_state_publisher namespace="$(arg namespace)" update_rate="50"/>
-  <!-- Initilizing thruster macro, might use another macro to achieve thrusters -->
-  <xacro:thruster_macro namespace="$(arg namespace)" thruster_id="0" mesh_scale="1">
-    <origin xyz="0.6650895 0.367385 0.828822" rpy="0 0 ${3*pi/4}"/>
+  <!-- Initilizing thruster macro, found in actuators.xacro -->
+  <xacro:thruster_macro namespace="$(arg namespace)" thruster_id="0" mesh_scale="${scale_factor}">
+    <origin xyz="${0.6650895*scale_factor} ${0.367385*scale_factor} ${0.828822*scale_factor}" rpy="0 0 ${3*pi/4}"/>
   </xacro:thruster_macro>
-  <xacro:thruster_macro namespace="$(arg namespace)" thruster_id="1" mesh_scale="1">
-    <origin xyz="0.665895 -0.367385 0.828822" rpy="0 0 ${-3*pi/4}"/>
+  <xacro:thruster_macro namespace="$(arg namespace)" thruster_id="1" mesh_scale="${scale_factor}">
+    <origin xyz="${0.665895*scale_factor} ${-0.367385*scale_factor} ${0.828822*scale_factor}" rpy="0 0 ${-3*pi/4}"/>
   </xacro:thruster_macro>
-  <!-- initilizing Sonar macro -->
-  <!--xacro:forward_multibeam_sonar_m450_130 namespace="$(arg namespace)" parent_link="$(arg namespace)/base_link" visualize="$(arg visualize)">
-    <origin xyz="-0.9 0 0.97" rpy="0 0 3.14159"/>
-  </xacro:forward_multibeam_sonar_m450_130-->
 <!-- kanskje prøve å etterligne denne https://waterlinked.com/shop/wl-21045-2-sonar-3d-15-689 -->
-  <xacro:sonar_3d
-    parent_link="$(arg namespace)/base_link"
-    namespace="$(arg namespace)"
-    visualize="$(arg visualize)"/>
+  <!-- Macro from sonar_snippets file -->
+<xacro:sonar_3d parent_link="$(arg namespace)/base_link" namespace="$(arg namespace)" scale_factor="${scale_factor}">
+    <origin xyz="${-0.8*scale_factor} 0 ${0.98*scale_factor}" rpy="0 0 ${pi}"/>
+</xacro:sonar_3d>
   <!-- imu sensor -->
   <link name= "imu_link">
@@ -136,5 +134,5 @@
       <child link= "imu_link" />
       <!-- <origin xyz= "0.55 0 3 " rpy= "0 0 0"/> -->
-      <origin xyz="0 0 0.81" rpy="0 0 0"/>
+      <origin xyz="0 0 ${0.81*scale_factor}" rpy="0 0 0"/>
   </joint>
   <gazebo reference="imu_link">
@@ -158,31 +156,24 @@
     </sensor>
   </gazebo>
-  <!-- Spawning in ArUco 5x5 marker -->
-  <link name="$(arg namespace)/aruco_marker">
-  <visual>
-    <origin xyz="0.25 0 0.41" rpy="${pi/2} 0 ${-pi/2}"/>
-    <geometry>
-      <mesh filename="file://$(find deep_ocean)/materials/textures/marker_5x5_0.dae" scale="0.6 0.6 0.6"/>
-    </geometry>
-  </visual>
-  </link>
-  <joint name="$(arg namespace)/aruco_joint" type="fixed">
-    <parent link="$(arg namespace)/base_link"/>
-    <child link="$(arg namespace)/aruco_marker"/>
-    <origin xyz="0 0 0" rpy="0 0 0"/>
-  </joint>
-  <!-- Spawning a calibration board of 7x10 dimension -->
-  <!-- <link name="$(arg namespace)/calibration_board">
-  <visual>
-    <origin xyz="-2 1 0.4" rpy="${pi/2} 0 ${-pi/2}"/>
-    <geometry>
-      <mesh filename="file://$(find deep_ocean)/materials/textures/checkerboard_7x10_bordered.dae" scale="0.6 0.6 0.6"/>
-    </geometry>
-  </visual>
-  </link>
-  <joint name="$(arg namespace)/checker_joint" type="fixed">
-    <parent link="$(arg namespace)/base_link"/>
-    <child link="$(arg namespace)/calibration_board"/>
-    <origin xyz="0 0 0" rpy="0 0 0"/>
-  </joint> -->
+    <!-- Spawning in ArUco 5x5 marker -->
+  <xacro:aruco_marker_5x5 namespace="$(arg namespace)" parent_link="$(arg namespace)/base_link" id="0" scale="${0.3*scale_factor}">
+    <origin xyz="${0.25*scale_factor} 0 ${0.66*scale_factor}" rpy="${pi/2} 0 ${-pi/2}"/>
+  </xacro:aruco_marker_5x5>
+    <!-- Spawning in ArUco 4x4 marker -->
+  <xacro:aruco_marker_4x4 namespace="$(arg namespace)" parent_link="$(arg namespace)/base_link" id="0" scale="${scale_factor}">
+    <origin xyz="${-0.8*scale_factor} ${0.5*scale_factor} ${0.97*scale_factor}" rpy="${pi/2} 0 ${-pi/2}"/>
+  </xacro:aruco_marker_4x4>
+  <xacro:aruco_marker_4x4 namespace="$(arg namespace)" parent_link="$(arg namespace)/base_link" id="1" scale="${scale_factor}">
+    <origin xyz="${-0.8*scale_factor} ${0.5*scale_factor} 0" rpy="${pi/2} 0 ${-pi/2}"/>
+  </xacro:aruco_marker_4x4>
+  <xacro:aruco_marker_4x4 namespace="$(arg namespace)" parent_link="$(arg namespace)/base_link" id="2" scale="${scale_factor}">
+    <origin xyz="${-0.8*scale_factor} ${-0.5*scale_factor} 0" rpy="${pi/2} 0 ${-pi/2}"/>
+  </xacro:aruco_marker_4x4>
+  <xacro:aruco_marker_4x4 namespace="$(arg namespace)" parent_link="$(arg namespace)/base_link" id="3" scale="${scale_factor}">
+    <origin xyz="${-0.8*scale_factor} ${-0.5*scale_factor} ${0.97*scale_factor}" rpy="${pi/2} 0 ${-pi/2}"/>
+  </xacro:aruco_marker_4x4>
+<!-- Example 3: Calibration board with custom ID -->
+<!-- <xacro:calibration_board namespace="$(arg namespace)" parent_link="$(arg namespace)/base_link" id="0" scale="1.0">
+  <origin xyz="-2 1 0.4" rpy="${pi/2} 0 ${-pi/2}"/>
+</xacro:calibration_board> -->
 </robot>

File: urdf/sonar_snippets.xacro (robot description, xacro)
@@ -129,9 +129,9 @@
   </xacro:macro>
   <!-- Macro a 3d depth sonar -->
-  <xacro:macro name="sonar_3d" params="parent_link namespace visualize:=true">
+<xacro:macro name="sonar_3d" params="parent_link namespace visualize:=true scale_factor:=1.0 *origin">
     <link name="${namespace}/sonar_3d_link">
       <visual>
         <geometry>
-          <box size="0.04 0.12 0.08"/>
+          <box size="${scale_factor*0.04} ${scale_factor*0.12} ${scale_factor*0.08}"/>
         </geometry>
         <material name="red">
@@ -142,9 +142,9 @@
         <mass value="0.0"/>
         <origin xyz="0 0 0"/>
-        <inertia ixx="0.1" ixy="0.0" ixz="0.0" iyy="0.1" iyz="0.0" izz="0.1"/>
+        <inertia ixx="${scale_factor*0.1}" ixy="0.0" ixz="0.0" iyy="${scale_factor*0.1}" iyz="0.0" izz="${scale_factor*0.1}"/>
       </inertial>
       <collision>
         <geometry>
-          <box size="0.04 0.12 0.08"/>
+          <box size="${scale_factor*0.04} ${scale_factor*0.12} ${scale_factor*0.08}"/>
         </geometry>
       </collision>
@@ -153,5 +153,5 @@
       <parent link="${parent_link}"/>
       <child link="${namespace}/sonar_3d_link"/>
-      <origin xyz="-0.8 0 1.02" rpy="0 0 3.14159"/>
+      <xacro:insert_block name="origin" />
     </joint>
     <link name="${namespace}/sonar_3d_optical_link"/>
@@ -175,6 +175,6 @@
             </image>
             <clip>
-              <near>0.1</near>
-              <far>5.0</far>
+              <near>${scale_factor*0.1}</near>
+              <far>${scale_factor*5.0}</far>
             </clip>
           </camera>
@@ -192,5 +192,5 @@
       </gazebo>
     </xacro:if>
-  </xacro:macro>
+</xacro:macro>
   <xacro:macro name="forward_looking_sonar"
     params="namespace suffix parent_link topic mass update_rate
