Commit message: Add files via upload

File: robots/rov_2d_sonar.xacro (robot description, xacro)
@@ -119,111 +119,11 @@
         </plugin>
     </gazebo>
-  <!-- imu sensor -->
-  <link name= "imu_link">
-      <visual>
-          <geometry>
-              <box size= "0.01 0.01 0.01" />
-          </geometry>
-          <material name= "red" >
-              <color rgba= "1 0 0 1" />
-          </material>
-      </visual>
-      <inertial>
-          <!-- <mass value= "0.39" /> -->
-          <mass value= "0.0" />
-          <origin xyz= "0 0 0" />
-          <inertia ixx= "0.1" ixy= "0.0" ixz= "0.0" iyy= "0.1" iyz= "0.0" izz= "0.1" />
-      </inertial>
-      <collision>
-          <geometry>
-              <box size= "0.01 0.01 0.01" />
-          </geometry>
-      </collision>
-  </link>
-  <joint name= "imu_joint" type= "fixed">
-      <parent link= "$(arg namespace)/base_link" />
-      <child link= "imu_link" />
-      <!-- <origin xyz= "0.55 0 3 " rpy= "0 0 0"/> -->
-      <origin xyz="0 0 0.81" rpy="0 0 0"/>
-  </joint>
-  <gazebo reference="imu_link">
-    <gravity>true</gravity>
-    <sensor name="imu_sensor" type="imu">
-      <always_on>true</always_on>
-      <update_rate>10</update_rate>
-      <visualize>true</visualize>
-      <topic>__default_topic__</topic>
-      <plugin filename="libgazebo_ros_imu_sensor.so" name="imu_plugin">
-        <topicName>imu</topicName>
-        <bodyName>imu_link</bodyName>
-        <updateRateHZ>10.0</updateRateHZ>
-        <gaussianNoise>0.0</gaussianNoise>
-        <xyzOffset>0 0 0</xyzOffset>
-        <rpyOffset>0 0 0</rpyOffset>
-        <frameName>imu_link</frameName>
-        <initialOrientationAsReference>false</initialOrientationAsReference>
-      </plugin>
-      <pose>0 0 0 0 0 0</pose>
-    </sensor>
-  </gazebo>
+    <!-- imu sensor -->
+    <xacro:imu_sensor parent_link="$(arg namespace)/base_link" namespace="$(arg namespace)">
+        <origin xyz="0 0 0.63" rpy="0 0 0"/>
+    </xacro:imu_sensor>
       <!-- camera -->
-    <link name= "camera_link">
-        <visual>
-            <geometry>
-                <box size= "0.1 0.1 0.1" />
-            </geometry>
-            <material name= "red" >
-                <color rgba= "1 0 0 1" />
-            </material>
-        </visual>
-        <inertial>
-            <mass value= "0.2" />
-            <origin xyz= "0 0 0" />
-            <inertia ixx= "0.1" ixy= "0.0" ixz= "0.0" iyy= "0.1" iyz= "0.0" izz= "0.1" />
-        </inertial>
-        <collision>
-            <geometry>
-                <box size= "0.1 0.1 0.1" />
-            </geometry>
-        </collision>
-    </link>
-    <joint name= "camera_joint" type= "fixed">
-        <parent link= "$(arg namespace)/base_link" />
-        <child link= "camera_link" />
-        <origin xyz="0.63 0 0.4" rpy="0 0 0"/>
-    </joint>
-    <link name= "camera_link_optical"></link>
-    <joint name= "camera_optical_joint" type= "fixed">
-        <parent link= "camera_link" />
-        <child link= "camera_link_optical" />
-        <origin xyz= "0 0 0 " rpy= "-1.57 0 -1.57"/>
-    </joint>
-    <gazebo reference= "camera_link">
-        <material>Gazebo/Red</material>
-        <sensor type= "camera" name= "camera_sensor">
-            <pose>0 0 0 0 0 0</pose>
-            <visualize>true</visualize>
-            <update_rate>30</update_rate>
-            <camera>
-                <horizontal_fov>1.047</horizontal_fov>
-                <image>
-                    <width>640</width>
-                    <height>480</height>
-                    <format>R8G8B8</format>
-                </image>
-                <clip>
-                    <near>0.1</near>
-                    <far>10</far>
-                </clip>
-            </camera>
-            <plugin name= "camera_controller" filename= "libgazebo_ros_camera.so" >
-                <frameName>camera_link_optical</frameName>
-                <alwaysOn>true</alwaysOn>
-                <updateRate>0.0</updateRate>
-                <cameraName>camera</cameraName>
-                <imageTopicName>image_raw</imageTopicName>
-                <cameraInfoTopicName>camera_info</cameraInfoTopicName>
-            </plugin>
-        </sensor>
-    </gazebo>
+    <xacro:camera_sensor parent_link="$(arg namespace)/base_link" namespace="$(arg namespace)">
+    <origin xyz="0.63 0 0.4" rpy="0 0 0"/>
+    </xacro:camera_sensor>
 </robot>

File: robots/rov_3d_sonar.xacro (robot description, xacro)
@@ -4,4 +4,5 @@
     <!-- Necessary for sensors -->
     <xacro:include filename="$(find deep_ocean)/urdf/sonar_snippets.xacro" />
+    <xacro:include filename="$(find deep_ocean)/urdf/sensor_snippets.xacro" />
     <!-- <xacro:include filename="$(find uuv_sensor_ros_plugins)/urdf/sensor_snippets.xacro"/> -->
     <!-- Necessary for thrusters -->
@@ -71,12 +72,4 @@
   </xacro:thruster_macro>
   <xacro:default_joint_state_publisher namespace="$(arg namespace)" update_rate="50"/>
-    <!-- initilizing Sonar macro -->
-  <!-- <xacro:forward_multibeam_sonar_m450_130 namespace="$(arg namespace)" parent_link="$(arg namespace)/base_link">
-    <origin xyz="0.63 0 0.63" rpy="0 0 0"/>
-  </xacro:forward_multibeam_sonar_m450_130> -->
-    <!-- mounting camera -->
-  <!--xacro:default_camera namespace="$(arg namespace)" parent_link="$(arg namespace)/base_link" suffix="">
-    <origin xyz="0.63 0 0.4" rpy="0 0.6 0"/>
-  </xacro:default_camera-->
     <gazebo>
         <plugin name="uuv_plugin" filename="libuuv_underwater_object_ros_plugin.so">
@@ -119,176 +112,15 @@
         </plugin>
     </gazebo>
-<!-- kanskje prøve å etterligne denne https://waterlinked.com/shop/wl-21045-2-sonar-3d-15-689 -->
-  <link name= "$(arg namespace)/depth_camera_link">
-      <visual>
-          <geometry>
-              <box size= "0.04 0.12 0.08" />
-          </geometry>
-          <material name= "red" >
-              <color rgba= "1 0 0 1" />
-          </material>
-      </visual>
-      <inertial>
-          <!-- <mass value= "0.39" /> -->
-          <mass value= "0.0" />
-          <origin xyz= "0 0 0" />
-          <inertia ixx= "0.1" ixy= "0.0" ixz= "0.0" iyy= "0.1" iyz= "0.0" izz= "0.1" />
-      </inertial>
-      <collision>
-          <geometry>
-              <box size= "0.04 0.12 0.08" />
-          </geometry>
-      </collision>
-  </link>
-    <joint name= "depth_camera_joint" type= "fixed">
-        <parent link= "$(arg namespace)/base_link" />
-        <child link= "$(arg namespace)/depth_camera_link" />
-        <!-- <origin xyz= "0.55 0 3 " rpy= "0 0 0"/> -->
+    <!-- kanskje prøve å etterligne denne https://waterlinked.com/shop/wl-21045-2-sonar-3d-15-689 -->
+    <xacro:sonar_3d parent_link="$(arg namespace)/base_link" namespace="$(arg namespace)" scale_factor="1">
         <origin xyz="0.63 0 0.63" rpy="0 0 0"/>
-    </joint>
-  <!-- optical link and joint for rviz -->
-  <link name= "$(arg namespace)/depth_camera_optical_link"></link>
-  <joint name= "depth_camera_optical_joint" type= "fixed">
-      <parent link= "$(arg namespace)/depth_camera_link" />
-      <child link= "$(arg namespace)/depth_camera_optical_link" />
-      <origin xyz= "0 0 0 " rpy= "-1.57 0 -1.57"/>
-  </joint>
-  <gazebo reference= "$(arg namespace)/depth_camera_link">
-      <material>Gazebo/Red</material>
-      <sensor name= "depth_camera_link" type= "depth">
-          <visualize>true</visualize>
-          <updateRate>10</updateRate>
-          <camera>
-              <horizontal_fov>1.57</horizontal_fov>
-              <vertical_fov>0.698</vertical_fov>
-              <image>
-                  <width>160</width>
-                  <height>100</height>
-              </image>
-              <clip>
-                  <near>0.1</near>
-                  <far>5.0</far>
-              </clip>
-          </camera>
-          <plugin name="depth_camera_sensor" filename="libgazebo_ros_openni_kinect.so">
-              <cameraName>depth_camera</cameraName>
-              <frameName>$(arg namespace)/depth_camera_optical_link</frameName>
-              <alwaysOn>true</alwaysOn>
-              <pointCloudTopicName>points</pointCloudTopicName>
-              <imageTopicName>rgb/image_raw</imageTopicName>
-              <depthImageTopicName>depth/image_raw</depthImageTopicName>
-              <cameraInfoTopicName>rgb/camera_info</cameraInfoTopicName>
-              <depthImageCameraInfoTopicName>depth/camera_info</depthImageCameraInfoTopicName>
-              <!-- <baseline>0.1</baseline> -->
-          </plugin>
-      </sensor>
-  </gazebo>
+    </xacro:sonar_3d>
   <!-- imu sensor -->
-  <link name= "imu_link">
-      <visual>
-          <geometry>
-              <box size= "0.01 0.01 0.01" />
-          </geometry>
-          <material name= "red" >
-              <color rgba= "1 0 0 1" />
-          </material>
-      </visual>
-      <inertial>
-          <!-- <mass value= "0.39" /> -->
-          <mass value= "0.0" />
-          <origin xyz= "0 0 0" />
-          <inertia ixx= "0.1" ixy= "0.0" ixz= "0.0" iyy= "0.1" iyz= "0.0" izz= "0.1" />
-      </inertial>
-      <collision>
-          <geometry>
-              <box size= "0.01 0.01 0.01" />
-          </geometry>
-      </collision>
-  </link>
-  <joint name= "imu_joint" type= "fixed">
-      <parent link= "$(arg namespace)/base_link" />
-      <child link= "imu_link" />
-      <!-- <origin xyz= "0.55 0 3 " rpy= "0 0 0"/> -->
-      <origin xyz="0 0 0.81" rpy="0 0 0"/>
-  </joint>
-  <gazebo reference="imu_link">
-    <gravity>true</gravity>
-    <sensor name="imu_sensor" type="imu">
-      <always_on>true</always_on>
-      <update_rate>10</update_rate>
-      <visualize>true</visualize>
-      <topic>__default_topic__</topic>
-      <plugin filename="libgazebo_ros_imu_sensor.so" name="imu_plugin">
-        <topicName>imu</topicName>
-        <bodyName>imu_link</bodyName>
-        <updateRateHZ>10.0</updateRateHZ>
-        <gaussianNoise>0.0</gaussianNoise>
-        <xyzOffset>0 0 0</xyzOffset>
-        <rpyOffset>0 0 0</rpyOffset>
-        <frameName>imu_link</frameName>
-        <initialOrientationAsReference>false</initialOrientationAsReference>
-      </plugin>
-      <pose>0 0 0 0 0 0</pose>
-    </sensor>
-  </gazebo>
+    <xacro:imu_sensor parent_link="$(arg namespace)/base_link" namespace="$(arg namespace)">
+        <origin xyz="0 0 0.63" rpy="0 0 0"/>
+    </xacro:imu_sensor>
       <!-- camera -->
-    <link name= "camera_link">
-        <visual>
-            <geometry>
-                <box size= "0.1 0.1 0.1" />
-            </geometry>
-            <material name= "red" >
-                <color rgba= "1 0 0 1" />
-            </material>
-        </visual>
-        <inertial>
-            <mass value= "0.2" />
-            <origin xyz= "0 0 0" />
-            <inertia ixx= "0.1" ixy= "0.0" ixz= "0.0" iyy= "0.1" iyz= "0.0" izz= "0.1" />
-        </inertial>
-        <collision>
-            <geometry>
-                <box size= "0.1 0.1 0.1" />
-            </geometry>
-        </collision>
-    </link>
-    <joint name= "camera_joint" type= "fixed">
-        <parent link= "$(arg namespace)/base_link" />
-        <child link= "camera_link" />
-        <origin xyz="0.63 0 0.4" rpy="0 0 0"/>
-    </joint>
-    <link name= "camera_link_optical"></link>
-    <joint name= "camera_optical_joint" type= "fixed">
-        <parent link= "camera_link" />
-        <child link= "camera_link_optical" />
-        <origin xyz= "0 0 0 " rpy= "-1.57 0 -1.57"/>
-    </joint>
-    <gazebo reference= "camera_link">
-        <material>Gazebo/Red</material>
-        <sensor type= "camera" name= "camera_sensor">
-            <pose>0 0 0 0 0 0</pose>
-            <visualize>true</visualize>
-            <update_rate>30</update_rate>
-            <camera>
-                <horizontal_fov>1.047</horizontal_fov>
-                <image>
-                    <width>640</width>
-                    <height>480</height>
-                    <format>R8G8B8</format>
-                </image>
-                <clip>
-                    <near>0.1</near>
-                    <far>10</far>
-                </clip>
-            </camera>
-            <plugin name= "camera_controller" filename= "libgazebo_ros_camera.so" >
-                <frameName>camera_link_optical</frameName>
-                <alwaysOn>true</alwaysOn>
-                <updateRate>0.0</updateRate>
-                <cameraName>camera</cameraName>
-                <imageTopicName>image_raw</imageTopicName>
-                <cameraInfoTopicName>camera_info</cameraInfoTopicName>
-            </plugin>
-        </sensor>
-    </gazebo>
+    <xacro:camera_sensor parent_link="$(arg namespace)/base_link" namespace="$(arg namespace)">
+    <origin xyz="0.63 0 0.4" rpy="0 0 0"/>
+    </xacro:camera_sensor>
 </robot>

File: robots/tms_2d_sonar.xacro (robot description, xacro)
@@ -96,51 +96,7 @@
   </gazebo>
   <!-- imu sensor -->
-  <link name= "imu_link">
-      <visual>
-          <geometry>
-              <box size= "0.01 0.01 0.01" />
-          </geometry>
-          <material name= "red" >
-              <color rgba= "1 0 0 1" />
-          </material>
-      </visual>
-      <inertial>
-          <!-- <mass value= "0.39" /> -->
-          <mass value= "0.0" />
-          <origin xyz= "0 0 0" />
-          <inertia ixx= "0.1" ixy= "0.0" ixz= "0.0" iyy= "0.1" iyz= "0.0" izz= "0.1" />
-      </inertial>
-      <collision>
-          <geometry>
-              <box size= "0.01 0.01 0.01" />
-          </geometry>
-      </collision>
-  </link>
-  <joint name= "imu_joint" type= "fixed">
-      <parent link= "$(arg namespace)/base_link" />
-      <child link= "imu_link" />
-      <!-- <origin xyz= "0.55 0 3 " rpy= "0 0 0"/> -->
+  <xacro:imu_sensor parent_link="$(arg namespace)/base_link" namespace="$(arg namespace)">
       <origin xyz="0 0 ${0.81*scale_factor}" rpy="0 0 0"/>
-  </joint>
-  <gazebo reference="imu_link">
-    <gravity>true</gravity>
-    <sensor name="imu_sensor" type="imu">
-      <always_on>true</always_on>
-      <update_rate>10</update_rate>
-      <visualize>true</visualize>
-      <topic>__default_topic__</topic>
-      <plugin filename="libgazebo_ros_imu_sensor.so" name="imu_plugin">
-        <topicName>imu</topicName>
-        <bodyName>imu_link</bodyName>
-        <updateRateHZ>10.0</updateRateHZ>
-        <gaussianNoise>0.0</gaussianNoise>
-        <xyzOffset>0 0 0</xyzOffset>
-        <rpyOffset>0 0 0</rpyOffset>
-        <frameName>imu_link</frameName>
-        <initialOrientationAsReference>false</initialOrientationAsReference>
-      </plugin>
-      <pose>0 0 0 0 0 0</pose>
-    </sensor>
-  </gazebo>
+  </xacro:imu_sensor>
   <xacro:default_joint_state_publisher namespace="$(arg namespace)" update_rate="50"/>
   <!-- Initilizing thruster macro, might use another macro to achieve thrusters -->

File: robots/tms_3d_sonar.xacro (robot description, xacro)
@@ -5,4 +5,5 @@
   <xacro:arg name="visualize" default="true"/>
   <xacro:include filename="$(find deep_ocean)/urdf/sonar_snippets.xacro" />
+  <xacro:include filename="$(find deep_ocean)/urdf/sensor_snippets.xacro" />
   <!-- Necessary for thruster_macro to work -->
   <xacro:include filename="$(find deep_ocean)/urdf/actuators.xacro" />
@@ -16,5 +17,5 @@
   <xacro:property name="fluid_density" value="1028"/>
   <!-- Scaling Factor for the TMS. Greater size means it's easier to dock -->
-  <xacro:property name="scale_factor" value="2"/> <!-- Change this to scale up/down -->
+  <xacro:property name="scale_factor" value="1.1"/> <!-- Change this to scale up/down -->
   <!-- Original Dimensions of the TMS -->
   <xacro:property name="size_x_orig" value="1.64"/>
@@ -105,70 +106,26 @@
 <!-- kanskje prøve å etterligne denne https://waterlinked.com/shop/wl-21045-2-sonar-3d-15-689 -->
   <!-- Macro from sonar_snippets file -->
-<xacro:sonar_3d parent_link="$(arg namespace)/base_link" namespace="$(arg namespace)" scale_factor="${scale_factor}">
-    <origin xyz="${-0.8*scale_factor} 0 ${0.98*scale_factor}" rpy="0 0 ${pi}"/>
-</xacro:sonar_3d>
+  <xacro:sonar_3d parent_link="$(arg namespace)/base_link" namespace="$(arg namespace)" scale_factor="${scale_factor}">
+      <origin xyz="${-0.8*scale_factor} 0 ${0.98*scale_factor}" rpy="0 0 ${pi}"/>
+  </xacro:sonar_3d>
   <!-- imu sensor -->
-  <link name= "imu_link">
-      <visual>
-          <geometry>
-              <box size= "0.01 0.01 0.01" />
-          </geometry>
-          <material name= "red" >
-              <color rgba= "1 0 0 1" />
-          </material>
-      </visual>
-      <inertial>
-          <!-- <mass value= "0.39" /> -->
-          <mass value= "0.0" />
-          <origin xyz= "0 0 0" />
-          <inertia ixx= "0.1" ixy= "0.0" ixz= "0.0" iyy= "0.1" iyz= "0.0" izz= "0.1" />
-      </inertial>
-      <collision>
-          <geometry>
-              <box size= "0.01 0.01 0.01" />
-          </geometry>
-      </collision>
-  </link>
-  <joint name= "imu_joint" type= "fixed">
-      <parent link= "$(arg namespace)/base_link" />
-      <child link= "imu_link" />
-      <!-- <origin xyz= "0.55 0 3 " rpy= "0 0 0"/> -->
+  <xacro:imu_sensor parent_link="$(arg namespace)/base_link" namespace="$(arg namespace)">
       <origin xyz="0 0 ${0.81*scale_factor}" rpy="0 0 0"/>
-  </joint>
-  <gazebo reference="imu_link">
-    <gravity>true</gravity>
-    <sensor name="imu_sensor" type="imu">
-      <always_on>true</always_on>
-      <update_rate>10</update_rate>
-      <visualize>true</visualize>
-      <topic>__default_topic__</topic>
-      <plugin filename="libgazebo_ros_imu_sensor.so" name="imu_plugin">
-        <topicName>imu</topicName>
-        <bodyName>imu_link</bodyName>
-        <updateRateHZ>10.0</updateRateHZ>
-        <gaussianNoise>0.0</gaussianNoise>
-        <xyzOffset>0 0 0</xyzOffset>
-        <rpyOffset>0 0 0</rpyOffset>
-        <frameName>imu_link</frameName>
-        <initialOrientationAsReference>false</initialOrientationAsReference>
-      </plugin>
-      <pose>0 0 0 0 0 0</pose>
-    </sensor>
-  </gazebo>
+  </xacro:imu_sensor>
     <!-- Spawning in ArUco 5x5 marker -->
-  <xacro:aruco_marker_5x5 namespace="$(arg namespace)" parent_link="$(arg namespace)/base_link" id="0" scale="${0.3*scale_factor}">
+  <xacro:aruco_marker_5x5 namespace="$(arg namespace)" parent_link="$(arg namespace)/base_link" id="0" scale="0.3">
     <origin xyz="${0.25*scale_factor} 0 ${0.66*scale_factor}" rpy="${pi/2} 0 ${-pi/2}"/>
   </xacro:aruco_marker_5x5>
     <!-- Spawning in ArUco 4x4 marker -->
-  <xacro:aruco_marker_4x4 namespace="$(arg namespace)" parent_link="$(arg namespace)/base_link" id="0" scale="${scale_factor}">
+  <xacro:aruco_marker_4x4 namespace="$(arg namespace)" parent_link="$(arg namespace)/base_link" id="0" scale="1">
     <origin xyz="${-0.8*scale_factor} ${0.5*scale_factor} ${0.97*scale_factor}" rpy="${pi/2} 0 ${-pi/2}"/>
   </xacro:aruco_marker_4x4>
-  <xacro:aruco_marker_4x4 namespace="$(arg namespace)" parent_link="$(arg namespace)/base_link" id="1" scale="${scale_factor}">
+  <xacro:aruco_marker_4x4 namespace="$(arg namespace)" parent_link="$(arg namespace)/base_link" id="1" scale="1">
     <origin xyz="${-0.8*scale_factor} ${0.5*scale_factor} 0" rpy="${pi/2} 0 ${-pi/2}"/>
   </xacro:aruco_marker_4x4>
-  <xacro:aruco_marker_4x4 namespace="$(arg namespace)" parent_link="$(arg namespace)/base_link" id="2" scale="${scale_factor}">
+  <xacro:aruco_marker_4x4 namespace="$(arg namespace)" parent_link="$(arg namespace)/base_link" id="2" scale="1">
     <origin xyz="${-0.8*scale_factor} ${-0.5*scale_factor} 0" rpy="${pi/2} 0 ${-pi/2}"/>
   </xacro:aruco_marker_4x4>
-  <xacro:aruco_marker_4x4 namespace="$(arg namespace)" parent_link="$(arg namespace)/base_link" id="3" scale="${scale_factor}">
+  <xacro:aruco_marker_4x4 namespace="$(arg namespace)" parent_link="$(arg namespace)/base_link" id="3" scale="1">
     <origin xyz="${-0.8*scale_factor} ${-0.5*scale_factor} ${0.97*scale_factor}" rpy="${pi/2} 0 ${-pi/2}"/>
   </xacro:aruco_marker_4x4>
