Commit message: Add files via upload

File: robots/rov_3d_sonar.xacro (robot description, xacro)
@@ -12,4 +12,5 @@
     <!-- Necessary for state publishing -->
     <xacro:include filename="$(find uuv_gazebo_ros_plugins)/urdf/misc.xacro" />
+    <xacro:include filename="$(find deep_ocean)/urdf/flashlight.xacro" />
     <!-- Fluid Density of Water (kg/m³) -->
     <xacro:property name="fluid_density" value="1028"/>
@@ -124,3 +125,6 @@
     <origin xyz="0.63 0 0.4" rpy="0 0 0"/>
     </xacro:camera_sensor>
+    <xacro:flashlight parent_link="$(arg namespace)/base_link" namespace="$(arg namespace)">
+    <origin xyz="0.63 0 0.5" rpy="0 -1.57 0"/>
+    </xacro:flashlight>
 </robot>

File: robots/tms_3d_sonar.xacro (robot description, xacro)
@@ -119,14 +119,14 @@
     <!-- Spawning in ArUco 4x4 marker -->
   <xacro:aruco_marker_4x4 namespace="$(arg namespace)" parent_link="$(arg namespace)/base_link" id="0" scale="1">
-    <origin xyz="${-0.8*scale_factor} ${0.5*scale_factor} ${0.97*scale_factor}" rpy="${pi/2} 0 ${-pi/2}"/>
+    <origin xyz="${-0.8*scale_factor} ${0.5*scale_factor} ${0.465*scale_factor}" rpy="${pi/2} 0 ${-pi/2}"/>
   </xacro:aruco_marker_4x4>
-  <xacro:aruco_marker_4x4 namespace="$(arg namespace)" parent_link="$(arg namespace)/base_link" id="1" scale="1">
+  <!-- <xacro:aruco_marker_4x4 namespace="$(arg namespace)" parent_link="$(arg namespace)/base_link" id="1" scale="1">
     <origin xyz="${-0.8*scale_factor} ${0.5*scale_factor} 0" rpy="${pi/2} 0 ${-pi/2}"/>
   </xacro:aruco_marker_4x4>
   <xacro:aruco_marker_4x4 namespace="$(arg namespace)" parent_link="$(arg namespace)/base_link" id="2" scale="1">
     <origin xyz="${-0.8*scale_factor} ${-0.5*scale_factor} 0" rpy="${pi/2} 0 ${-pi/2}"/>
-  </xacro:aruco_marker_4x4>
+  </xacro:aruco_marker_4x4> -->
   <xacro:aruco_marker_4x4 namespace="$(arg namespace)" parent_link="$(arg namespace)/base_link" id="3" scale="1">
-    <origin xyz="${-0.8*scale_factor} ${-0.5*scale_factor} ${0.97*scale_factor}" rpy="${pi/2} 0 ${-pi/2}"/>
+    <origin xyz="${-0.8*scale_factor} ${-0.5*scale_factor} ${0.465*scale_factor}" rpy="${pi/2} 0 ${-pi/2}"/>
   </xacro:aruco_marker_4x4>
 <!-- Example 3: Calibration board with custom ID -->

File: urdf/sonar_snippets.xacro (robot description, xacro)
@@ -43,27 +43,4 @@
         <geometry>
           <mesh filename="file://$(find uuv_sensor_ros_plugins)/meshes/m450-130.dae" scale="0.5 0.5 0.5"/>
-        </geometry>
-      </visual>
-    </xacro:multibeam_sonar>
-  </xacro:macro>
-  <xacro:macro name="forward_multibeam_p900" params="namespace parent_link *origin">
-    <xacro:multibeam_sonar
-      namespace="${namespace}"
-      suffix=""
-      parent_link="${parent_link}"
-      topic="sonar"
-      mass="0.02"
-      update_rate="15"
-      samples="512"
-      fov="1.0"
-      range_min="1.0"
-      range_max="100.0"
-      range_stddev="0.027"
-      mesh="">
-      <inertia ixx="0.00001" ixy="0.0" ixz="0.0" iyy="0.00001" iyz="0.0" izz="0.00001" />
-      <xacro:insert_block name="origin" />
-      <visual>
-        <geometry>
-          <mesh filename="file://$(find uuv_sensor_ros_plugins)/meshes/p900.dae" scale="1 1 1"/>
         </geometry>
       </visual>
@@ -193,63 +170,3 @@
     </xacro:if>
 </xacro:macro>
-  <xacro:macro name="forward_looking_sonar"
-    params="namespace suffix parent_link topic mass update_rate
-      samples fov width height *inertia *origin">
-    <!-- Sensor link -->
-    <link name="${namespace}/forward_sonar${suffix}_link">
-      <inertial>
-        <xacro:insert_block name="inertia" />
-        <mass value="${mass}" />
-        <origin xyz="0 0 0" rpy="0 0 0" />
-      </inertial>
-      <visual>
-        <geometry>
-          <mesh filename="file://$(find uuv_sensor_ros_plugins)/meshes/oe14-372.dae" scale="1 1 1"/>
-        </geometry>
-      </visual>
-      <xacro:no_collision/>
-    </link>
-    <joint name="${namespace}_forward_sonar${suffix}_joint" type="revolute">
-      <xacro:insert_block name="origin" />
-      <parent link="${parent_link}" />
-      <child link="${namespace}/forward_sonar${suffix}_link" />
-      <limit upper="0" lower="0" effort="0" velocity="0" />
-      <axis xyz="1 0 0"/>
-    </joint>
-    <gazebo reference="${namespace}/forward_sonar${suffix}_link">
-      <sensor name="${namespace}/image_sonar" type="depth">
-        <camera>
-		  <horizontal_fov>${fov}</horizontal_fov>
-          <image>
-		    <width>${width}</width>
-		    <height>${height}</height>
-            <format>R8G8B8</format>
-          </image>
-          <clip>
-            <near>0.1</near>
-            <far>17</far>
-          </clip>
-          <save enabled="true">
-            <path>/tmp/camera</path>
-          </save>
-        </camera>
-	    <!--plugin filename="libimage_sonar_ros_plugin.so" name="forward_sonar${suffix}_controller">
-		  <topicName>${topic}</topicName>
-          <frameName>forward_sonar${suffix}_optical_frame</frameName>
-      </plugin-->
-      <plugin name="depth_camera_plugin" filename="gazebo_ros_image_sonar.hh">
-        <topicName>/sonar_camera</topicName>
-        <frameName>sonar_camera_frame</frameName>
-      </plugin>
-        <always_on>true</always_on>
-	    <update_rate>${update_rate}</update_rate>
-      </sensor>
-    </gazebo>
-	<joint name="${namespace}/forward_sonar${suffix}_joint" type="fixed">
-      <origin xyz="0 0 0" rpy="${-pi/2} 0 ${-pi/2}"/>
-      <parent link="${namespace}/forward_sonar${suffix}_link"/>
-      <child link="${namespace}/forward_sonar${suffix}_optical_frame"/>
-    </joint>
-	<link name="${namespace}/forward_sonar${suffix}_optical_frame"/>
-  </xacro:macro>
 </robot>

Commit message: Add files via upload

File: robots/rov_3d_sonar.xacro (robot description, xacro)
@@ -2,52 +2,52 @@
 <robot name="rov" xmlns:xacro="http://www.ros.org/wiki/xacro">
   <xacro:arg name="namespace" default="rov"/>
-    <!-- Necessary for sensors -->
-    <xacro:include filename="$(find deep_ocean)/urdf/sonar_snippets.xacro" />
-    <xacro:include filename="$(find deep_ocean)/urdf/sensor_snippets.xacro" />
-    <!-- <xacro:include filename="$(find uuv_sensor_ros_plugins)/urdf/sensor_snippets.xacro"/> -->
-    <!-- Necessary for thrusters -->
-    <xacro:include filename="$(find deep_ocean)/urdf/actuators.xacro" />
-    <xacro:include filename="$(find uuv_descriptions)/urdf/common.urdf.xacro" />
-    <xacro:include filename="$(find deep_ocean)/urdf/thruster_snippets.xacro" />
-    <!-- Necessary for state publishing -->
-    <xacro:include filename="$(find uuv_gazebo_ros_plugins)/urdf/misc.xacro" />
-    <xacro:include filename="$(find deep_ocean)/urdf/flashlight.xacro" />
-    <!-- Fluid Density of Water (kg/m³) -->
-    <xacro:property name="fluid_density" value="1028"/>
-    <!-- Hardcoded Dimensions from the Collision Mesh -->
-    <xacro:property name="size_y" value="0.833"/> <!-- Width -->
-    <xacro:property name="size_x" value="1.25"/>  <!-- Length -->
-    <xacro:property name="size_z" value="0.77"/>  <!-- Height -->
-    <!-- Mass of the ROV -->
-    <xacro:property name="mass" value="326"/>
-    <!-- Compute Volume to Ensure Neutral Buoyancy -->
-    <xacro:property name="volume" value="${mass / fluid_density}"/>
-    <!-- Center of Buoyancy Adjusted -->
-    <xacro:property name="cob_z" value="${0.5 * size_z}"/>
-    <!-- Inertia Calculation -->
-    <xacro:property name="ixx" value="${(1/12) * mass * (size_x * size_x + size_z * size_z)}"/>
-    <xacro:property name="iyy" value="${(1/12) * mass * (size_y * size_y + size_z * size_z)}"/>
-    <xacro:property name="izz" value="${(1/12) * mass * (size_y * size_y + size_x * size_x)}"/>
-    <!-- Define Base Link -->
-    <link name="$(arg namespace)/base_link">
-        <inertial>
-            <mass value="${mass}"/>
-            <origin xyz="0 0 0" rpy="0 0 0"/>
-            <inertia ixx="${ixx}" ixy="0.0" ixz="0.0" iyy="${iyy}" iyz="0.0" izz="${izz}"/>
-        </inertial>
-        <!-- Visual Representation -->
-        <visual>
-            <geometry>
-                <mesh filename="package://deep_ocean/meshes/rov_visual.dae" scale="1 1 1"/>
-            </geometry>
-        </visual>
-        <!-- Collision Geometry -->
-        <collision>
-            <origin xyz="0 0 0" rpy="0 0 0"/>
-            <geometry>
-                <mesh filename="package://deep_ocean/meshes/rov_collision.stl" scale="1 1 1"/>
-            </geometry>
-        </collision>
-    </link>
+  <xacro:arg name="inertial_reference_frame" default="world"/>
+  <!-- Necessary for sensors -->
+  <xacro:include filename="$(find deep_ocean)/urdf/sonar_snippets.xacro" />
+  <xacro:include filename="$(find deep_ocean)/urdf/sensor_snippets.xacro" />
+  <xacro:include filename="$(find uuv_sensor_ros_plugins)/urdf/dvl_snippets.xacro" />
+  <!-- Necessary for thrusters -->
+  <xacro:include filename="$(find deep_ocean)/urdf/actuators.xacro" />
+  <xacro:include filename="$(find uuv_descriptions)/urdf/common.urdf.xacro" />
+  <xacro:include filename="$(find deep_ocean)/urdf/thruster_snippets.xacro" />
+  <!-- Necessary for state publishing -->
+  <xacro:include filename="$(find uuv_gazebo_ros_plugins)/urdf/misc.xacro" />
+  <!-- Fluid Density of Water (kg/m³) -->
+  <xacro:property name="fluid_density" value="1028"/>
+  <!-- Hardcoded Dimensions from the Collision Mesh -->
+  <xacro:property name="size_y" value="0.833"/> <!-- Width -->
+  <xacro:property name="size_x" value="1.25"/>  <!-- Length -->
+  <xacro:property name="size_z" value="0.77"/>  <!-- Height -->
+  <!-- Mass of the ROV -->
+  <xacro:property name="mass" value="326"/>
+  <!-- Compute Volume to Ensure Neutral Buoyancy -->
+  <xacro:property name="volume" value="${mass / fluid_density}"/>
+  <!-- Center of Buoyancy Adjusted -->
+  <xacro:property name="cob_z" value="${0.5 * size_z}"/>
+  <!-- Inertia Calculation -->
+  <xacro:property name="ixx" value="${(1/12) * mass * (size_x * size_x + size_z * size_z)}"/>
+  <xacro:property name="iyy" value="${(1/12) * mass * (size_y * size_y + size_z * size_z)}"/>
+  <xacro:property name="izz" value="${(1/12) * mass * (size_y * size_y + size_x * size_x)}"/>
+  <!-- Define Base Link -->
+  <link name="$(arg namespace)/base_link">
+      <inertial>
+          <mass value="${mass}"/>
+          <origin xyz="0 0 0" rpy="0 0 0"/>
+          <inertia ixx="${ixx}" ixy="0.0" ixz="0.0" iyy="${iyy}" iyz="0.0" izz="${izz}"/>
+      </inertial>
+      <!-- Visual Representation -->
+      <visual>
+          <geometry>
+              <mesh filename="package://deep_ocean/meshes/rov_visual.dae" scale="1 1 1"/>
+          </geometry>
+      </visual>
+      <!-- Collision Geometry -->
+      <collision>
+          <origin xyz="0 0 0" rpy="0 0 0"/>
+          <geometry>
+              <mesh filename="package://deep_ocean/meshes/rov_collision.stl" scale="1 1 1"/>
+          </geometry>
+      </collision>
+  </link>
     <!-- Initiating thrusters from UUV -->
   <xacro:thruster_macro namespace="$(arg namespace)" thruster_id="0">
@@ -73,58 +73,70 @@
   </xacro:thruster_macro>
   <xacro:default_joint_state_publisher namespace="$(arg namespace)" update_rate="50"/>
-    <gazebo>
-        <plugin name="uuv_plugin" filename="libuuv_underwater_object_ros_plugin.so">
-            <fluid_density>${fluid_density}</fluid_density>
-            <flow_velocity_topic>hydrodynamics/current_velocity</flow_velocity_topic>
-            <debug>0</debug>
-            <link name="$(arg namespace)/base_link">
-                <neutrally_buoyant>1</neutrally_buoyant>  <!-- Ensures mass and volume decide float/sink -->
-                <volume>${volume}</volume>
-                <box>
-                    <width>${size_y}</width>
-                    <length>${size_x}</length>
-                    <height>${size_z}</height>
-                </box>
-                <center_of_buoyancy>0 0 ${cob_z}</center_of_buoyancy>
-                <!-- Hydrodynamic Model using Fossen type -->
-                <hydrodynamic_model>
-                    <type>fossen</type>
-                    <!-- Rough Added Mass Estimation -->
-                    <added_mass>
-                        ${0.1 * mass}  0  0  0  0  0
-                        0  ${0.1 * mass}  0  0  0  0
-                        0  0  ${0.1 * mass}  0  0  0
-                        0  0  0  ${0.05 * mass}  0  0
-                        0  0  0  0  ${0.05 * mass}  0
-                        0  0  0  0  0  ${0.05 * mass}
-                    </added_mass>
-                    <!-- Rough Linear Damping Estimation -->
-                    <linear_damping>
-                        ${-100 * size_y} ${-100 * size_x} ${-100 * size_z}
-                        ${-40 * size_z} ${-40 * size_x} ${-40 * size_y}
-                    </linear_damping>
-                    <!-- Rough Quadratic Damping Estimation -->
-                    <quadratic_damping>
-                        ${-120 * size_y} ${-120 * size_x} ${-120 * size_z}
-                        ${-50 * size_z} ${-50 * size_x} ${-50 * size_y}
-                    </quadratic_damping>
-                </hydrodynamic_model>
-            </link>
-        </plugin>
-    </gazebo>
+  <gazebo>
+      <plugin name="uuv_plugin" filename="libuuv_underwater_object_ros_plugin.so">
+          <fluid_density>${fluid_density}</fluid_density>
+          <flow_velocity_topic>hydrodynamics/current_velocity</flow_velocity_topic>
+          <debug>0</debug>
+          <link name="$(arg namespace)/base_link">
+              <neutrally_buoyant>1</neutrally_buoyant>  <!-- Ensures mass and volume decide float/sink -->
+              <volume>${volume}</volume>
+              <box>
+                  <width>${size_y}</width>
+                  <length>${size_x}</length>
+                  <height>${size_z}</height>
+              </box>
+              <center_of_buoyancy>0 0 ${cob_z}</center_of_buoyancy>
+              <!-- Hydrodynamic Model using Fossen type -->
+              <hydrodynamic_model>
+                  <type>fossen</type>
+                  <!-- Rough Added Mass Estimation -->
+                  <added_mass>
+                      ${0.1 * mass}  0  0  0  0  0
+                      0  ${0.1 * mass}  0  0  0  0
+                      0  0  ${0.1 * mass}  0  0  0
+                      0  0  0  ${0.05 * mass}  0  0
+                      0  0  0  0  ${0.05 * mass}  0
+                      0  0  0  0  0  ${0.05 * mass}
+                  </added_mass>
+                  <!-- Rough Linear Damping Estimation -->
+                  <linear_damping>
+                      ${-100 * size_y} ${-100 * size_x} ${-100 * size_z}
+                      ${-40 * size_z} ${-40 * size_x} ${-40 * size_y}
+                  </linear_damping>
+                  <!-- Rough Quadratic Damping Estimation -->
+                  <quadratic_damping>
+                      ${-120 * size_y} ${-120 * size_x} ${-120 * size_z}
+                      ${-50 * size_z} ${-50 * size_x} ${-50 * size_y}
+                  </quadratic_damping>
+              </hydrodynamic_model>
+          </link>
+      </plugin>
+      <!-- Odometry for the PID -->
+      <plugin name="p3d_base_controller" filename="libgazebo_ros_p3d.so">
+        <robotNamespace>/$(arg namespace)</robotNamespace>
+        <bodyName>$(arg namespace)/base_link</bodyName>
+        <topicName>pose_gt</topicName>
+        <frameName>world</frameName>  <!-- or "odom" if using a local frame -->
+        <updateRate>30</updateRate>
+      </plugin>
+  </gazebo>
     <!-- kanskje prøve å etterligne denne https://waterlinked.com/shop/wl-21045-2-sonar-3d-15-689 -->
-    <xacro:sonar_3d parent_link="$(arg namespace)/base_link" namespace="$(arg namespace)" scale_factor="1">
-        <origin xyz="0.63 0 0.63" rpy="0 0 0"/>
-    </xacro:sonar_3d>
-  <!-- imu sensor -->
-    <xacro:imu_sensor parent_link="$(arg namespace)/base_link" namespace="$(arg namespace)">
-        <origin xyz="0 0 0.63" rpy="0 0 0"/>
-    </xacro:imu_sensor>
-      <!-- camera -->
-    <xacro:camera_sensor parent_link="$(arg namespace)/base_link" namespace="$(arg namespace)">
+  <xacro:sonar_3d parent_link="$(arg namespace)/base_link" namespace="$(arg namespace)" scale_factor="1">
+    <origin xyz="0.63 0 0.63" rpy="0 0 0"/>
+  </xacro:sonar_3d>
+<!-- imu sensor -->
+  <xacro:imu_sensor parent_link="$(arg namespace)/base_link" namespace="$(arg namespace)">
+    <origin xyz="0 0 0.63" rpy="0 0 0"/>
+  </xacro:imu_sensor>
+    <!-- camera -->
+  <xacro:camera_sensor parent_link="$(arg namespace)/base_link" namespace="$(arg namespace)">
     <origin xyz="0.63 0 0.4" rpy="0 0 0"/>
-    </xacro:camera_sensor>
-    <xacro:flashlight parent_link="$(arg namespace)/base_link" namespace="$(arg namespace)">
-    <origin xyz="0.63 0 0.5" rpy="0 -1.57 0"/>
-    </xacro:flashlight>
+  </xacro:camera_sensor>
+  <!-- DVL from UUV simulator -->
+  <!-- <xacro:default_dvl_macro
+    namespace="$(arg namespace)"
+    parent_link="$(arg namespace)/base_link"
+    inertial_reference_frame="$(arg inertial_reference_frame)">
+    <origin xyz="-0.6 0 0" rpy="0 ${0.5*pi} 0"/>
+  </xacro:default_dvl_macro>  -->
 </robot>

File: robots/tms_3d_sonar.xacro (robot description, xacro)
@@ -27,5 +27,5 @@
   <xacro:property name="size_z" value="${size_z_orig * scale_factor}"/>
   <!-- Mass (Scaled) -->
-  <xacro:property name="mass" value="${550 * (scale_factor * scale_factor * scale_factor)}"/>
+  <xacro:property name="mass" value="${550 * scale_factor}"/>
   <!-- Volume (to ensure neutral buoyancy) -->
   <xacro:property name="volume" value="${mass / fluid_density}"/>
