Commit message: Add files via upload

File: robots/tms_3d_sonar.xacro (robot description, xacro)
@@ -17,5 +17,5 @@
   <xacro:property name="fluid_density" value="1028"/>
   <!-- Scaling Factor for the TMS. Greater size means it's easier to dock -->
-  <xacro:property name="scale_factor" value="1.1"/> <!-- Change this to scale up/down -->
+  <xacro:property name="scale_factor" value="1.4"/> <!-- Change this to scale up/down -->
   <!-- Original Dimensions of the TMS -->
   <xacro:property name="size_x_orig" value="1.64"/>
@@ -115,5 +115,5 @@
     <!-- Spawning in ArUco 5x5 marker -->
   <xacro:aruco_marker_5x5 namespace="$(arg namespace)" parent_link="$(arg namespace)/base_link" id="0" scale="0.3">
-    <origin xyz="${0.25*scale_factor} 0 ${0.66*scale_factor}" rpy="${pi/2} 0 ${-pi/2}"/>
+    <origin xyz="${0.24*scale_factor} 0 ${0.66*scale_factor}" rpy="${pi/2} 0 ${-pi/2}"/>
   </xacro:aruco_marker_5x5>
     <!-- Spawning in ArUco 4x4 marker -->

Commit message: Add files via upload

File: robots/tms_3d_sonar.xacro (robot description, xacro)
@@ -115,5 +115,5 @@
     <!-- Spawning in ArUco 5x5 marker -->
   <xacro:aruco_marker_5x5 namespace="$(arg namespace)" parent_link="$(arg namespace)/base_link" id="0" scale="0.3">
-    <origin xyz="${0.24*scale_factor} 0 ${0.66*scale_factor}" rpy="${pi/2} 0 ${-pi/2}"/>
+    <origin xyz="${0.24*scale_factor} 0 ${0.5*scale_factor}" rpy="${pi/2} 0 ${-pi/2}"/>
   </xacro:aruco_marker_5x5>
     <!-- Spawning in ArUco 4x4 marker -->

Commit message: Add files via upload

File: robots/tms_3d_sonar.xacro (robot description, xacro)
@@ -27,5 +27,5 @@
   <xacro:property name="size_z" value="${size_z_orig * scale_factor}"/>
   <!-- Mass (Scaled) -->
-  <xacro:property name="mass" value="${550 * (scale_factor * scale_factor * scale_factor)}"/>
+  <xacro:property name="mass" value="${550}"/>
   <!-- Volume (to ensure neutral buoyancy) -->
   <xacro:property name="volume" value="${mass / fluid_density}"/>

Commit message: Add files via upload
same as Slightly-cleaner-package, but with tms scaling of 1.3

File: robots/tms_3d_sonar.xacro (robot description, xacro)
@@ -17,5 +17,5 @@
   <xacro:property name="fluid_density" value="1028"/>
   <!-- Scaling Factor for the TMS. Greater size means it's easier to dock -->
-  <xacro:property name="scale_factor" value="1.4"/> <!-- Change this to scale up/down -->
+  <xacro:property name="scale_factor" value="1.3"/> <!-- Change this to scale up/down -->
   <!-- Original Dimensions of the TMS -->
   <xacro:property name="size_x_orig" value="1.64"/>
@@ -39,5 +39,5 @@
     <inertial>
       <mass value="${mass}"/>
-      <origin xyz="0 0 0" rpy="0 0 3.14159"/>5
+      <origin xyz="0 0 0" rpy="0 0 3.14159"/>
       <inertia ixx="${ixx}" ixy="0.0" ixz="0.0" iyy="${iyy}" iyz="0.0" izz="${izz}"/>
     </inertial>
@@ -114,10 +114,10 @@
   </xacro:imu_sensor>
     <!-- Spawning in ArUco 5x5 marker -->
-  <xacro:aruco_marker_5x5 namespace="$(arg namespace)" parent_link="$(arg namespace)/base_link" id="0" scale="0.3">
-    <origin xyz="${0.24*scale_factor} 0 ${0.5*scale_factor}" rpy="${pi/2} 0 ${-pi/2}"/>
+  <xacro:aruco_marker_5x5 namespace="$(arg namespace)" parent_link="$(arg namespace)/base_link" id="0" scale="0.30">
+    <origin xyz="${0.24*scale_factor} 0 ${0.48*scale_factor}" rpy="${pi/2} 0 ${-pi/2}"/>
   </xacro:aruco_marker_5x5>
     <!-- Spawning in ArUco 4x4 marker -->
   <xacro:aruco_marker_4x4 namespace="$(arg namespace)" parent_link="$(arg namespace)/base_link" id="0" scale="1">
-    <origin xyz="${-0.8*scale_factor} ${0.5*scale_factor} ${0.465*scale_factor}" rpy="${pi/2} 0 ${-pi/2}"/>
+    <origin xyz="${-0.8*scale_factor} ${0.5*scale_factor} ${0.485*scale_factor}" rpy="${pi/2} 0 ${-pi/2}"/>
   </xacro:aruco_marker_4x4>
   <!-- <xacro:aruco_marker_4x4 namespace="$(arg namespace)" parent_link="$(arg namespace)/base_link" id="1" scale="1">
@@ -125,8 +125,8 @@
   </xacro:aruco_marker_4x4>
   <xacro:aruco_marker_4x4 namespace="$(arg namespace)" parent_link="$(arg namespace)/base_link" id="2" scale="1">
-    <origin xyz="${-0.8*scale_factor} ${-0.5*scale_factor} 0" rpy="${pi/2} 0 ${-pi/2}"/>
+    <origin xyz="${-0.8*scale_factor} ${-0.5*scale_factor} ${0.465*scale_factor}" rpy="${pi/2} 0 ${-pi/2}"/>
   </xacro:aruco_marker_4x4> -->
   <xacro:aruco_marker_4x4 namespace="$(arg namespace)" parent_link="$(arg namespace)/base_link" id="3" scale="1">
-    <origin xyz="${-0.8*scale_factor} ${-0.5*scale_factor} ${0.465*scale_factor}" rpy="${pi/2} 0 ${-pi/2}"/>
+    <origin xyz="${-0.8*scale_factor} ${-0.5*scale_factor} ${0.485*scale_factor}" rpy="${pi/2} 0 ${-pi/2}"/>
   </xacro:aruco_marker_4x4>
 <!-- Example 3: Calibration board with custom ID -->
