Commit message: Add files via upload

File: urdf_xacro_files/sensors_and_actuators/sensor_snippets.xacro (robot description, xacro)
@@ -53,20 +53,17 @@
     <link name="${namespace}/camera_link">
         <visual>
-        <geometry>
-            <box size="0.1 0.1 0.1" />
-        </geometry>
-        <material name="red">
-            <color rgba="1 0 0 1" />
-        </material>
+            <geometry>
+                <mesh filename="file://$(find deep_ocean)/meshes/exploreHD_camera.dae" />
+            </geometry>
         </visual>
         <inertial>
-        <mass value="0.2" />
-        <origin xyz="0 0 0" />
+            <mass value="0.2" />
+            <origin xyz="0 0 0" />
         <inertia ixx="0.1" ixy="0.0" ixz="0.0" iyy="0.1" iyz="0.0" izz="0.1" />
         </inertial>
         <collision>
-        <geometry>
-            <box size="0.1 0.1 0.1" />
-        </geometry>
+            <geometry>
+                <box size="0.1 0.1 0.1" />
+            </geometry>
         </collision>
     </link>
@@ -91,6 +88,6 @@
             <horizontal_fov>1.047</horizontal_fov>
             <image>
-            <width>1280</width>
-            <height>720</height>
+            <width>1920</width>
+            <height>1080</height>
             <format>R8G8B8</format>
             </image>

File: urdf_xacro_files/sensors_and_actuators/sonar_snippets.xacro (robot description, xacro)
@@ -31,8 +31,8 @@
       mass="0.0001"
       update_rate="25"
-      samples="100"
+      samples="768"
       fov="2.27"
       range_min="1.0"
-      range_max="10.0"
+      range_max="100.0"
       range_stddev="0.027"
       mesh=""
@@ -106,5 +106,5 @@
   </xacro:macro>
   <!-- Macro a 3d depth sonar -->
-<xacro:macro name="sonar_3d" params="parent_link namespace visualize:=true scale_factor:=1.0 *origin">
+<xacro:macro name="sonar_3d" params="parent_link namespace scale_factor:=1.0 *origin">
     <link name="${namespace}/sonar_3d_link">
       <visual>
@@ -138,35 +138,33 @@
       <origin xyz="0 0 0" rpy="-1.57 0 -1.57"/>
     </joint>
-    <xacro:if value="${visualize}">
-      <gazebo reference="${namespace}/sonar_3d_link">
-        <material>Gazebo/Red</material>
-        <sensor name="sonar_3d_sensor" type="depth">
-          <visualize>true</visualize>
-          <updateRate>10</updateRate>
-          <camera>
-            <horizontal_fov>1.57</horizontal_fov>
-            <vertical_fov>0.698</vertical_fov>
-            <image>
-              <width>160</width>
-              <height>100</height>
-            </image>
-            <clip>
-              <near>0.01</near>
-              <far>10.0</far>     <!-- Change the length of field of view-->
-            </clip>
-          </camera>
-          <plugin name="sonar_3d_plugin" filename="libgazebo_ros_openni_kinect.so">
-            <cameraName>${namespace}/sonar_3d</cameraName>
-            <frameName>${namespace}/sonar_3d_optical_link</frameName>
-            <alwaysOn>true</alwaysOn>
-            <pointCloudTopicName>points</pointCloudTopicName>
-            <imageTopicName>rgb/image_raw</imageTopicName>
-            <depthImageTopicName>depth/image_raw</depthImageTopicName>
-            <cameraInfoTopicName>rgb/camera_info</cameraInfoTopicName>
-            <depthImageCameraInfoTopicName>depth/camera_info</depthImageCameraInfoTopicName>
-          </plugin>
-        </sensor>
-      </gazebo>
-    </xacro:if>
+    <gazebo reference="${namespace}/sonar_3d_link">
+      <material>Gazebo/Red</material>
+      <sensor name="sonar_3d_sensor" type="depth">
+        <visualize>true</visualize>
+        <updateRate>10</updateRate>
+        <camera>
+          <horizontal_fov>1.57</horizontal_fov>
+          <vertical_fov>0.698</vertical_fov>
+          <image>
+            <width>160</width>
+            <height>100</height>
+          </image>
+          <clip>
+            <near>0.01</near>
+            <far>10.0</far>     <!-- Change the length of field of view-->
+          </clip>
+        </camera>
+        <plugin name="sonar_3d_plugin" filename="libgazebo_ros_openni_kinect.so">
+          <cameraName>${namespace}/sonar_3d</cameraName>
+          <frameName>${namespace}/sonar_3d_optical_link</frameName>
+          <alwaysOn>true</alwaysOn>
+          <pointCloudTopicName>points</pointCloudTopicName>
+          <imageTopicName>rgb/image_raw</imageTopicName>
+          <depthImageTopicName>depth/image_raw</depthImageTopicName>
+          <cameraInfoTopicName>rgb/camera_info</cameraInfoTopicName>
+          <depthImageCameraInfoTopicName>depth/camera_info</depthImageCameraInfoTopicName>
+        </plugin>
+      </sensor>
+    </gazebo>
 </xacro:macro>
 </robot>
