Commit message: Add files via upload

File: urdf_xacro_files/robots/tms_3d_sonar.xacro (robot description, xacro)
@@ -132,5 +132,5 @@
 <!-- Example 3: Calibration board with custom ID -->
 <!-- <xacro:calibration_board namespace="$(arg namespace)" parent_link="$(arg namespace)/base_link" id="0" scale="1.0">
-  <origin xyz="-2 1 0.4" rpy="${pi/2} 0 ${-pi/2}"/>
+  <origin xyz="-2 -8 0.4" rpy="1.37 0.15 -1.44"/>
 </xacro:calibration_board> -->
 </robot>

File: urdf_xacro_files/sensors_and_actuators/sensor_snippets.xacro (robot description, xacro)
@@ -54,5 +54,5 @@
         <visual>
             <geometry>
-                <mesh filename="file://$(find deep_ocean)/meshes/exploreHD_camera.dae" />
+                <mesh filename="file://$(find deep_ocean)/meshes/exploreHD_camera.stl" />
             </geometry>
         </visual>
@@ -83,5 +83,5 @@
         <sensor type="camera" name="camera_sensor">
         <pose>0 0 0 0 0 0</pose>
-        <visualize>true</visualize>
+        <!-- <visualize>true</visualize> -->
         <update_rate>30</update_rate>
         <camera>

File: urdf_xacro_files/sensors_and_actuators/sonar_snippets.xacro (robot description, xacro)
@@ -142,5 +142,5 @@
       <sensor name="sonar_3d_sensor" type="depth">
         <visualize>true</visualize>
-        <updateRate>10</updateRate>
+        <updateRate>5</updateRate>
         <camera>
           <horizontal_fov>1.57</horizontal_fov>
@@ -151,6 +151,6 @@
           </image>
           <clip>
-            <near>0.01</near>
-            <far>10.0</far>     <!-- Change the length of field of view-->
+            <near>0.02</near>
+            <far>15.0</far>     <!-- Change the length of field of view-->
           </clip>
         </camera>
