Commit message: Add files via upload

File: urdf_xacro_files/robots/rov_2d_sonar.xacro (robot description, xacro)
@@ -4,4 +4,5 @@
     <!-- Necessary for sensors -->
     <xacro:include filename="$(find deep_ocean)/urdf_xacro_files/sensors_and_actuators/sonar_snippets.xacro" />
+    <xacro:include filename="$(find deep_ocean)/urdf_xacro_files/sensors_and_actuators/sensor_snippets.xacro" />
     <!-- <xacro:include filename="$(find uuv_sensor_ros_plugins)/urdf/sensor_snippets.xacro"/> -->
     <!-- Necessary for thrusters -->

File: urdf_xacro_files/robots/tms_2d_sonar.xacro (robot description, xacro)
@@ -3,6 +3,7 @@
   <!-- Necessary for sonar to work -->
   <xacro:arg name="namespace" default="tms"/>
-  <xacro:arg name="visualize" default="true"/>
+  <xacro:arg name="visualize" default="false"/>
   <xacro:include filename="$(find deep_ocean)/urdf_xacro_files/sensors_and_actuators/sonar_snippets.xacro" />
+  <xacro:include filename="$(find deep_ocean)/urdf_xacro_files/sensors_and_actuators/sensor_snippets.xacro" />
   <!-- Necessary for thruster_macro to work -->
   <xacro:include filename="$(find deep_ocean)/urdf_xacro_files/sensors_and_actuators/actuators.xacro" />
@@ -16,5 +17,5 @@
   <xacro:property name="fluid_density" value="1028"/>
   <!-- Scaling Factor for the TMS. Greater size means it's easier to dock -->
-  <xacro:property name="scale_factor" value="1"/> <!-- Change this to scale up/down -->
+  <xacro:property name="scale_factor" value="1.3"/> <!-- Change this to scale up/down -->
   <!-- Original Dimensions of the TMS -->
   <xacro:property name="size_x_orig" value="1.64"/>
@@ -26,5 +27,5 @@
   <xacro:property name="size_z" value="${size_z_orig * scale_factor}"/>
   <!-- Mass (Scaled) -->
-  <xacro:property name="mass" value="${550 * (scale_factor * scale_factor * scale_factor)}"/>
+  <xacro:property name="mass" value="${550}"/>
   <!-- Volume (to ensure neutral buoyancy) -->
   <xacro:property name="volume" value="${mass / fluid_density}"/>
@@ -116,15 +117,15 @@
   </xacro:aruco_marker_5x5>
     <!-- Spawning in ArUco 4x4 marker -->
-  <xacro:aruco_marker_4x4 namespace="$(arg namespace)" parent_link="$(arg namespace)/base_link" id="0" scale="${scale_factor}">
-    <origin xyz="${-0.8*scale_factor} ${0.5*scale_factor} ${0.97*scale_factor}" rpy="${pi/2} 0 ${-pi/2}"/>
+  <xacro:aruco_marker_4x4 namespace="$(arg namespace)" parent_link="$(arg namespace)/base_link" id="0" scale="${1}">
+    <origin xyz="${-0.8*scale_factor} ${0.5*scale_factor} ${0.485*scale_factor}" rpy="${pi/2} 0 ${-pi/2}"/>
   </xacro:aruco_marker_4x4>
-  <xacro:aruco_marker_4x4 namespace="$(arg namespace)" parent_link="$(arg namespace)/base_link" id="1" scale="${scale_factor}">
+  <!-- <xacro:aruco_marker_4x4 namespace="$(arg namespace)" parent_link="$(arg namespace)/base_link" id="1" scale="${1}">
     <origin xyz="${-0.8*scale_factor} ${0.5*scale_factor} 0" rpy="${pi/2} 0 ${-pi/2}"/>
-  </xacro:aruco_marker_4x4>
-  <xacro:aruco_marker_4x4 namespace="$(arg namespace)" parent_link="$(arg namespace)/base_link" id="2" scale="${scale_factor}">
+  </xacro:aruco_marker_4x4> -->
+  <!-- <xacro:aruco_marker_4x4 namespace="$(arg namespace)" parent_link="$(arg namespace)/base_link" id="2" scale="${1}">
     <origin xyz="${-0.8*scale_factor} ${-0.5*scale_factor} 0" rpy="${pi/2} 0 ${-pi/2}"/>
-  </xacro:aruco_marker_4x4>
-  <xacro:aruco_marker_4x4 namespace="$(arg namespace)" parent_link="$(arg namespace)/base_link" id="3" scale="${scale_factor}">
-    <origin xyz="${-0.8*scale_factor} ${-0.5*scale_factor} ${0.97*scale_factor}" rpy="${pi/2} 0 ${-pi/2}"/>
+  </xacro:aruco_marker_4x4> -->
+  <xacro:aruco_marker_4x4 namespace="$(arg namespace)" parent_link="$(arg namespace)/base_link" id="3" scale="${1}">
+    <origin xyz="${-0.8*scale_factor} ${-0.5*scale_factor} ${0.485*scale_factor}" rpy="${pi/2} 0 ${-pi/2}"/>
   </xacro:aruco_marker_4x4>
 </robot>

File: urdf_xacro_files/sensors_and_actuators/sensor_snippets.xacro (robot description, xacro)
@@ -88,4 +88,8 @@
             <horizontal_fov>1.047</horizontal_fov>
             <image>
+            <!-- <width>1280</width>
+            <height>720</height> -->
+            <!-- <width>640</width>
+            <height>480</height> -->
             <width>1920</width>
             <height>1080</height>

File: urdf_xacro_files/sensors_and_actuators/sonar_snippets.xacro (robot description, xacro)
@@ -23,5 +23,5 @@
   </xacro:macro>
   <!-- Inspired by m450-130: http://www.blueview.com/products/2d-imaging-sonar/m900-series/ -->
-  <xacro:macro name="forward_multibeam_sonar_m450_130" params="namespace parent_link visualize:=true *origin">
+  <xacro:macro name="forward_multibeam_sonar_m450_130" params="namespace parent_link visualize:=false *origin">
     <xacro:multibeam_sonar
       namespace="${namespace}"
@@ -141,5 +141,5 @@
       <material>Gazebo/Red</material>
       <sensor name="sonar_3d_sensor" type="depth">
-        <visualize>true</visualize>
+        <!-- <visualize>true</visualize> -->
         <updateRate>5</updateRate>
         <camera>

Commit message: Add files via upload

File: urdf_xacro_files/robots/rov_2d_sonar.xacro (robot description, xacro)
@@ -4,5 +4,4 @@
     <!-- Necessary for sensors -->
     <xacro:include filename="$(find deep_ocean)/urdf_xacro_files/sensors_and_actuators/sonar_snippets.xacro" />
-    <xacro:include filename="$(find deep_ocean)/urdf_xacro_files/sensors_and_actuators/sensor_snippets.xacro" />
     <!-- <xacro:include filename="$(find uuv_sensor_ros_plugins)/urdf/sensor_snippets.xacro"/> -->
     <!-- Necessary for thrusters -->

File: urdf_xacro_files/robots/rov_3d_sonar.xacro (robot description, xacro)
@@ -74,42 +74,50 @@
   <xacro:default_joint_state_publisher namespace="$(arg namespace)" update_rate="50"/>
     <gazebo>
-        <plugin name="uuv_plugin" filename="libuuv_underwater_object_ros_plugin.so">
-            <fluid_density>${fluid_density}</fluid_density>
-            <flow_velocity_topic>hydrodynamics/current_velocity</flow_velocity_topic>
-            <debug>0</debug>
-            <link name="$(arg namespace)/base_link">
-                <neutrally_buoyant>1</neutrally_buoyant>  <!-- Ensures mass and volume decide float/sink -->
-                <volume>${volume}</volume>
-                <box>
-                    <width>${size_y}</width>
-                    <length>${size_x}</length>
-                    <height>${size_z}</height>
-                </box>
-                <center_of_buoyancy>0 0 ${cob_z}</center_of_buoyancy>
-                <!-- Hydrodynamic Model using Fossen type -->
-                <hydrodynamic_model>
-                    <type>fossen</type>
-                    <!-- Rough Added Mass Estimation -->
-                    <added_mass>
-                        ${0.1 * mass}  0  0  0  0  0
-                        0  ${0.1 * mass}  0  0  0  0
-                        0  0  ${0.1 * mass}  0  0  0
-                        0  0  0  ${0.05 * mass}  0  0
-                        0  0  0  0  ${0.05 * mass}  0
-                        0  0  0  0  0  ${0.05 * mass}
-                    </added_mass>
-                    <!-- Rough Linear Damping Estimation -->
-                    <linear_damping>
-                        ${-100 * size_y} ${-100 * size_x} ${-100 * size_z}
-                        ${-40 * size_z} ${-40 * size_x} ${-40 * size_y}
-                    </linear_damping>
-                    <!-- Rough Quadratic Damping Estimation -->
-                    <quadratic_damping>
-                        ${-120 * size_y} ${-120 * size_x} ${-120 * size_z}
-                        ${-50 * size_z} ${-50 * size_x} ${-50 * size_y}
-                    </quadratic_damping>
-                </hydrodynamic_model>
-            </link>
-        </plugin>
+      <plugin name="uuv_plugin" filename="libuuv_underwater_object_ros_plugin.so">
+        <fluid_density>${fluid_density}</fluid_density>
+        <flow_velocity_topic>hydrodynamics/current_velocity</flow_velocity_topic>
+        <debug>0</debug>
+        <link name="$(arg namespace)/base_link">
+            <neutrally_buoyant>1</neutrally_buoyant>  <!-- Ensures mass and volume decide float/sink -->
+            <volume>${volume}</volume>
+            <box>
+                <width>${size_y}</width>
+                <length>${size_x}</length>
+                <height>${size_z}</height>
+            </box>
+            <center_of_buoyancy>0 0 ${cob_z}</center_of_buoyancy>
+            <!-- Hydrodynamic Model using Fossen type -->
+            <hydrodynamic_model>
+                <type>fossen</type>
+                <!-- Rough Added Mass Estimation -->
+                <added_mass>
+                    ${0.1 * mass}  0  0  0  0  0
+                    0  ${0.1 * mass}  0  0  0  0
+                    0  0  ${0.1 * mass}  0  0  0
+                    0  0  0  ${0.05 * mass}  0  0
+                    0  0  0  0  ${0.05 * mass}  0
+                    0  0  0  0  0  ${0.05 * mass}
+                </added_mass>
+                <!-- Rough Linear Damping Estimation -->
+                <linear_damping>
+                    ${-100 * size_y} ${-100 * size_x} ${-100 * size_z}
+                    ${-40 * size_z} ${-40 * size_x} ${-40 * size_y}
+                </linear_damping>
+                <!-- Rough Quadratic Damping Estimation -->
+                <quadratic_damping>
+                    ${-120 * size_y} ${-120 * size_x} ${-120 * size_z}
+                    ${-50 * size_z} ${-50 * size_x} ${-50 * size_y}
+                </quadratic_damping>
+            </hydrodynamic_model>
+        </link>
+      </plugin>
+      <!-- Odometry for the PID -->
+      <plugin name="p3d_base_controller" filename="libgazebo_ros_p3d.so">
+        <robotNamespace>/$(arg namespace)</robotNamespace>
+        <bodyName>$(arg namespace)/base_link</bodyName>
+        <topicName>pose_gt</topicName>
+        <frameName>world</frameName>  <!-- or "odom" if using a local frame -->
+        <updateRate>30</updateRate>
+      </plugin>
     </gazebo>
     <!-- kanskje prøve å etterligne denne https://waterlinked.com/shop/wl-21045-2-sonar-3d-15-689 -->

File: urdf_xacro_files/robots/tms_2d_sonar.xacro (robot description, xacro)
@@ -3,7 +3,6 @@
   <!-- Necessary for sonar to work -->
   <xacro:arg name="namespace" default="tms"/>
-  <xacro:arg name="visualize" default="false"/>
+  <xacro:arg name="visualize" default="true"/>
   <xacro:include filename="$(find deep_ocean)/urdf_xacro_files/sensors_and_actuators/sonar_snippets.xacro" />
-  <xacro:include filename="$(find deep_ocean)/urdf_xacro_files/sensors_and_actuators/sensor_snippets.xacro" />
   <!-- Necessary for thruster_macro to work -->
   <xacro:include filename="$(find deep_ocean)/urdf_xacro_files/sensors_and_actuators/actuators.xacro" />
@@ -17,5 +16,5 @@
   <xacro:property name="fluid_density" value="1028"/>
   <!-- Scaling Factor for the TMS. Greater size means it's easier to dock -->
-  <xacro:property name="scale_factor" value="1.3"/> <!-- Change this to scale up/down -->
+  <xacro:property name="scale_factor" value="1"/> <!-- Change this to scale up/down -->
   <!-- Original Dimensions of the TMS -->
   <xacro:property name="size_x_orig" value="1.64"/>
@@ -27,5 +26,5 @@
   <xacro:property name="size_z" value="${size_z_orig * scale_factor}"/>
   <!-- Mass (Scaled) -->
-  <xacro:property name="mass" value="${550}"/>
+  <xacro:property name="mass" value="${550 * (scale_factor * scale_factor * scale_factor)}"/>
   <!-- Volume (to ensure neutral buoyancy) -->
   <xacro:property name="volume" value="${mass / fluid_density}"/>
@@ -117,15 +116,15 @@
   </xacro:aruco_marker_5x5>
     <!-- Spawning in ArUco 4x4 marker -->
-  <xacro:aruco_marker_4x4 namespace="$(arg namespace)" parent_link="$(arg namespace)/base_link" id="0" scale="${1}">
-    <origin xyz="${-0.8*scale_factor} ${0.5*scale_factor} ${0.485*scale_factor}" rpy="${pi/2} 0 ${-pi/2}"/>
+  <xacro:aruco_marker_4x4 namespace="$(arg namespace)" parent_link="$(arg namespace)/base_link" id="0" scale="${scale_factor}">
+    <origin xyz="${-0.8*scale_factor} ${0.5*scale_factor} ${0.97*scale_factor}" rpy="${pi/2} 0 ${-pi/2}"/>
   </xacro:aruco_marker_4x4>
-  <!-- <xacro:aruco_marker_4x4 namespace="$(arg namespace)" parent_link="$(arg namespace)/base_link" id="1" scale="${1}">
+  <xacro:aruco_marker_4x4 namespace="$(arg namespace)" parent_link="$(arg namespace)/base_link" id="1" scale="${scale_factor}">
     <origin xyz="${-0.8*scale_factor} ${0.5*scale_factor} 0" rpy="${pi/2} 0 ${-pi/2}"/>
-  </xacro:aruco_marker_4x4> -->
-  <!-- <xacro:aruco_marker_4x4 namespace="$(arg namespace)" parent_link="$(arg namespace)/base_link" id="2" scale="${1}">
+  </xacro:aruco_marker_4x4>
+  <xacro:aruco_marker_4x4 namespace="$(arg namespace)" parent_link="$(arg namespace)/base_link" id="2" scale="${scale_factor}">
     <origin xyz="${-0.8*scale_factor} ${-0.5*scale_factor} 0" rpy="${pi/2} 0 ${-pi/2}"/>
-  </xacro:aruco_marker_4x4> -->
-  <xacro:aruco_marker_4x4 namespace="$(arg namespace)" parent_link="$(arg namespace)/base_link" id="3" scale="${1}">
-    <origin xyz="${-0.8*scale_factor} ${-0.5*scale_factor} ${0.485*scale_factor}" rpy="${pi/2} 0 ${-pi/2}"/>
+  </xacro:aruco_marker_4x4>
+  <xacro:aruco_marker_4x4 namespace="$(arg namespace)" parent_link="$(arg namespace)/base_link" id="3" scale="${scale_factor}">
+    <origin xyz="${-0.8*scale_factor} ${-0.5*scale_factor} ${0.97*scale_factor}" rpy="${pi/2} 0 ${-pi/2}"/>
   </xacro:aruco_marker_4x4>
 </robot>

File: urdf_xacro_files/sensors_and_actuators/sensor_snippets.xacro (robot description, xacro)
@@ -88,8 +88,4 @@
             <horizontal_fov>1.047</horizontal_fov>
             <image>
-            <!-- <width>1280</width>
-            <height>720</height> -->
-            <!-- <width>640</width>
-            <height>480</height> -->
             <width>1920</width>
             <height>1080</height>

File: urdf_xacro_files/sensors_and_actuators/sonar_snippets.xacro (robot description, xacro)
@@ -23,5 +23,5 @@
   </xacro:macro>
   <!-- Inspired by m450-130: http://www.blueview.com/products/2d-imaging-sonar/m900-series/ -->
-  <xacro:macro name="forward_multibeam_sonar_m450_130" params="namespace parent_link visualize:=false *origin">
+  <xacro:macro name="forward_multibeam_sonar_m450_130" params="namespace parent_link visualize:=true *origin">
     <xacro:multibeam_sonar
       namespace="${namespace}"
@@ -141,5 +141,5 @@
       <material>Gazebo/Red</material>
       <sensor name="sonar_3d_sensor" type="depth">
-        <!-- <visualize>true</visualize> -->
+        <visualize>true</visualize>
         <updateRate>5</updateRate>
         <camera>
