Commit message: Add files via upload

File: urdf_xacro_files/robots/rov_2d_sonar.xacro (robot description, xacro)
@@ -73,12 +73,8 @@
   </xacro:thruster_macro>
   <xacro:default_joint_state_publisher namespace="$(arg namespace)" update_rate="50"/>
-    <!-- initilizing Sonar macro -->
+    <!-- initilizing Sonar macro from UUV -->
   <xacro:forward_multibeam_sonar_m450_130 namespace="$(arg namespace)" parent_link="$(arg namespace)/base_link" visualize="$(arg visualize)">
     <origin xyz="0.63 0 0.63" rpy="0 0 0"/>
   </xacro:forward_multibeam_sonar_m450_130>
-    <!-- mounting camera -->
-  <!--xacro:default_camera namespace="$(arg namespace)" parent_link="$(arg namespace)/base_link" suffix="">
-    <origin xyz="0.63 0 0.4" rpy="0 0.6 0"/>
-  </xacro:default_camera-->
     <gazebo>
         <plugin name="uuv_plugin" filename="libuuv_underwater_object_ros_plugin.so">

File: urdf_xacro_files/robots/rov_3d_sonar.xacro (robot description, xacro)
@@ -12,5 +12,4 @@
     <!-- Necessary for state publishing -->
     <xacro:include filename="$(find uuv_gazebo_ros_plugins)/urdf/misc.xacro" />
-    <xacro:include filename="$(find deep_ocean)/urdf_xacro_files/sensors_and_actuators/flashlight.xacro" />
     <!-- Fluid Density of Water (kg/m³) -->
     <xacro:property name="fluid_density" value="1028"/>
@@ -74,57 +73,62 @@
   <xacro:default_joint_state_publisher namespace="$(arg namespace)" update_rate="50"/>
     <gazebo>
-        <plugin name="uuv_plugin" filename="libuuv_underwater_object_ros_plugin.so">
-            <fluid_density>${fluid_density}</fluid_density>
-            <flow_velocity_topic>hydrodynamics/current_velocity</flow_velocity_topic>
-            <debug>0</debug>
-            <link name="$(arg namespace)/base_link">
-                <neutrally_buoyant>1</neutrally_buoyant>  <!-- Ensures mass and volume decide float/sink -->
-                <volume>${volume}</volume>
-                <box>
-                    <width>${size_y}</width>
-                    <length>${size_x}</length>
-                    <height>${size_z}</height>
-                </box>
-                <center_of_buoyancy>0 0 ${cob_z}</center_of_buoyancy>
-                <!-- Hydrodynamic Model using Fossen type -->
-                <hydrodynamic_model>
-                    <type>fossen</type>
-                    <!-- Rough Added Mass Estimation -->
-                    <added_mass>
-                        ${0.1 * mass}  0  0  0  0  0
-                        0  ${0.1 * mass}  0  0  0  0
-                        0  0  ${0.1 * mass}  0  0  0
-                        0  0  0  ${0.05 * mass}  0  0
-                        0  0  0  0  ${0.05 * mass}  0
-                        0  0  0  0  0  ${0.05 * mass}
-                    </added_mass>
-                    <!-- Rough Linear Damping Estimation -->
-                    <linear_damping>
-                        ${-100 * size_y} ${-100 * size_x} ${-100 * size_z}
-                        ${-40 * size_z} ${-40 * size_x} ${-40 * size_y}
-                    </linear_damping>
-                    <!-- Rough Quadratic Damping Estimation -->
-                    <quadratic_damping>
-                        ${-120 * size_y} ${-120 * size_x} ${-120 * size_z}
-                        ${-50 * size_z} ${-50 * size_x} ${-50 * size_y}
-                    </quadratic_damping>
-                </hydrodynamic_model>
-            </link>
-        </plugin>
+      <plugin name="uuv_plugin" filename="libuuv_underwater_object_ros_plugin.so">
+        <fluid_density>${fluid_density}</fluid_density>
+        <flow_velocity_topic>hydrodynamics/current_velocity</flow_velocity_topic>
+        <debug>0</debug>
+        <link name="$(arg namespace)/base_link">
+          <neutrally_buoyant>1</neutrally_buoyant>  <!-- Ensures mass and volume decide float/sink -->
+          <volume>${volume}</volume>
+          <box>
+              <width>${size_y}</width>
+              <length>${size_x}</length>
+              <height>${size_z}</height>
+          </box>
+          <center_of_buoyancy>0 0 ${cob_z}</center_of_buoyancy>
+          <!-- Hydrodynamic Model using Fossen type -->
+          <hydrodynamic_model>
+              <type>fossen</type>
+              <!-- Rough Added Mass Estimation -->
+              <added_mass>
+                  ${0.1 * mass}  0  0  0  0  0
+                  0  ${0.1 * mass}  0  0  0  0
+                  0  0  ${0.1 * mass}  0  0  0
+                  0  0  0  ${0.05 * mass}  0  0
+                  0  0  0  0  ${0.05 * mass}  0
+                  0  0  0  0  0  ${0.05 * mass}
+              </added_mass>
+              <!-- Rough Linear Damping Estimation -->
+              <linear_damping>
+                  ${-100 * size_y} ${-100 * size_x} ${-100 * size_z}
+                  ${-40 * size_z} ${-40 * size_x} ${-40 * size_y}
+              </linear_damping>
+              <!-- Rough Quadratic Damping Estimation -->
+              <quadratic_damping>
+                  ${-120 * size_y} ${-120 * size_x} ${-120 * size_z}
+                  ${-50 * size_z} ${-50 * size_x} ${-50 * size_y}
+              </quadratic_damping>
+          </hydrodynamic_model>
+        </link>
+      </plugin>
+      <!-- Odometry for the PID -->
+      <plugin name="p3d_base_controller" filename="libgazebo_ros_p3d.so">
+        <robotNamespace>/$(arg namespace)</robotNamespace>
+        <bodyName>$(arg namespace)/base_link</bodyName>
+        <topicName>pose_gt</topicName>
+        <frameName>world</frameName>
+        <updateRate>30</updateRate>
+      </plugin>
     </gazebo>
-    <!-- kanskje prøve å etterligne denne https://waterlinked.com/shop/wl-21045-2-sonar-3d-15-689 -->
+    <!-- 3D sonar -->
     <xacro:sonar_3d parent_link="$(arg namespace)/base_link" namespace="$(arg namespace)" scale_factor="1">
         <origin xyz="0.63 0 0.63" rpy="0 0 0"/>
     </xacro:sonar_3d>
-  <!-- imu sensor -->
+    <!-- imu sensor -->
     <xacro:imu_sensor parent_link="$(arg namespace)/base_link" namespace="$(arg namespace)">
         <origin xyz="0 0 0.63" rpy="0 0 0"/>
     </xacro:imu_sensor>
-      <!-- camera -->
+    <!-- camera -->
     <xacro:camera_sensor parent_link="$(arg namespace)/base_link" namespace="$(arg namespace)">
     <origin xyz="0.63 0 0.4" rpy="0 0 0"/>
     </xacro:camera_sensor>
-    <xacro:flashlight parent_link="$(arg namespace)/base_link" namespace="$(arg namespace)">
-    <origin xyz="0.63 0 0.5" rpy="0 -1.57 0"/>
-    </xacro:flashlight>
 </robot>

File: urdf_xacro_files/robots/tms_2d_sonar.xacro (robot description, xacro)
@@ -101,5 +101,5 @@
   </xacro:imu_sensor>
   <xacro:default_joint_state_publisher namespace="$(arg namespace)" update_rate="50"/>
-  <!-- Initilizing thruster macro, might use another macro to achieve thrusters -->
+  <!-- Initilizing thruster macro -->
   <xacro:thruster_macro namespace="$(arg namespace)" thruster_id="0" mesh_scale="${scale_factor}">
     <origin xyz="${0.6650895*scale_factor} ${0.367385*scale_factor} ${0.828822*scale_factor}" rpy="0 0 ${3*pi/4}"/>
@@ -120,10 +120,4 @@
     <origin xyz="${-0.8*scale_factor} ${0.5*scale_factor} ${0.485*scale_factor}" rpy="${pi/2} 0 ${-pi/2}"/>
   </xacro:aruco_marker_4x4>
-  <!-- <xacro:aruco_marker_4x4 namespace="$(arg namespace)" parent_link="$(arg namespace)/base_link" id="1" scale="${1}">
-    <origin xyz="${-0.8*scale_factor} ${0.5*scale_factor} 0" rpy="${pi/2} 0 ${-pi/2}"/>
-  </xacro:aruco_marker_4x4> -->
-  <!-- <xacro:aruco_marker_4x4 namespace="$(arg namespace)" parent_link="$(arg namespace)/base_link" id="2" scale="${1}">
-    <origin xyz="${-0.8*scale_factor} ${-0.5*scale_factor} 0" rpy="${pi/2} 0 ${-pi/2}"/>
-  </xacro:aruco_marker_4x4> -->
   <xacro:aruco_marker_4x4 namespace="$(arg namespace)" parent_link="$(arg namespace)/base_link" id="3" scale="${1}">
     <origin xyz="${-0.8*scale_factor} ${-0.5*scale_factor} ${0.485*scale_factor}" rpy="${pi/2} 0 ${-pi/2}"/>

File: urdf_xacro_files/robots/tms_3d_sonar.xacro (robot description, xacro)
@@ -104,5 +104,4 @@
     <origin xyz="${0.665895*scale_factor} ${-0.367385*scale_factor} ${0.828822*scale_factor}" rpy="0 0 ${-3*pi/4}"/>
   </xacro:thruster_macro>
-<!-- kanskje prøve å etterligne denne https://waterlinked.com/shop/wl-21045-2-sonar-3d-15-689 -->
   <!-- Macro from sonar_snippets file -->
   <xacro:sonar_3d parent_link="$(arg namespace)/base_link" namespace="$(arg namespace)" scale_factor="${scale_factor}">
@@ -121,14 +120,7 @@
     <origin xyz="${-0.8*scale_factor} ${0.5*scale_factor} ${0.485*scale_factor}" rpy="${pi/2} 0 ${-pi/2}"/>
   </xacro:aruco_marker_4x4>
-  <!-- <xacro:aruco_marker_4x4 namespace="$(arg namespace)" parent_link="$(arg namespace)/base_link" id="1" scale="1">
-    <origin xyz="${-0.8*scale_factor} ${0.5*scale_factor} 0" rpy="${pi/2} 0 ${-pi/2}"/>
-  </xacro:aruco_marker_4x4>
-  <xacro:aruco_marker_4x4 namespace="$(arg namespace)" parent_link="$(arg namespace)/base_link" id="2" scale="1">
-    <origin xyz="${-0.8*scale_factor} ${-0.5*scale_factor} ${0.465*scale_factor}" rpy="${pi/2} 0 ${-pi/2}"/>
-  </xacro:aruco_marker_4x4> -->
   <xacro:aruco_marker_4x4 namespace="$(arg namespace)" parent_link="$(arg namespace)/base_link" id="3" scale="1">
     <origin xyz="${-0.8*scale_factor} ${-0.5*scale_factor} ${0.485*scale_factor}" rpy="${pi/2} 0 ${-pi/2}"/>
   </xacro:aruco_marker_4x4>
-<!-- Example 3: Calibration board with custom ID -->
 <!-- <xacro:calibration_board namespace="$(arg namespace)" parent_link="$(arg namespace)/base_link" id="0" scale="1.0">
   <origin xyz="-2 -8 0.4" rpy="1.37 0.15 -1.44"/>
